File: electronics/template_one_unit/template_one_unit.kicad_pcb (KiCad board)
At the start: 2 copper layers, 2 parts

Commit message: finished one unit cell
Parts:
- added J1: LEFT_TOP, mill-max:PC_pin_nail_head_6092, F.Cu at (142.0, 63.0)
- added J2: LEFT_BOT, mill-max:PC_pin_nail_head_6092, F.Cu at (142.0, 78.0)
- added J3: RIGHT_TOP, mill-max:PC_pin_nail_head_6092, F.Cu at (157.0, 63.0)
- added J4: RIGHT_BOT, mill-max:PC_pin_nail_head_6092, F.Cu at (157.0, 78.0)
- N1: value 20200610 -> 20201118; moved to B.Cu
- N2: moved to B.Cu
- moved N1 21.1 mm to (149.1, 73.5)
- moved N2 21.1 mm to (149.7, 69.6), turned to 180 degrees
Other:
- board outline added: 19 x 19 mm
