File: electronics/proto_2by2/proto_2by2.kicad_pcb (KiCad board)
At the start: 2 copper layers, 34 x 34 mm, 8 parts, among them J1 1, J2 2, J3 3, J4 4, J5 5, J6 6

Commit message: updated versionnumber
Parts:
- added U1: KOSMOS_protoarea_6pin, SquantorProto:proto-TH-0254-KOSGRID-2X2-P020SQ-H010, F.Cu at (157.0, 78.0)
- N1: value 20201120 -> 20201122
Connections:
- J1 pad 1: Net-(J1-Pad1) -> /1
- J2 pad 1: Net-(J1-Pad1) -> /2
- J3 pad 1: Net-(J1-Pad1) -> /3
- J4 pad 1: Net-(J1-Pad1) -> /4
- J5 pad 1: Net-(J1-Pad1) -> /5
- J6 pad 1: Net-(J1-Pad1) -> /6

Commit message: placed and routed 2 by 2 grid
Parts:
- removed N1: 20201122, SquantorLabels:Label_Generic
- removed N2: OHWLOGO, Symbol:OSHW-Symbol_6.7x6mm_SilkScreen
Routing:
- net /5: track 0.00 -> 2.64 mm
- net /2: track 0.00 -> 2.64 mm
- net /6: track 0.00 -> 2.40 mm
- net /1: track 0.00 -> 2.40 mm
- net /4: track 0.00 -> 2.40 mm
- net /3: track 0.00 -> 2.40 mm
