File: electronics/template_1by2_high_density_XN/template_1by2_high_density_XN.kicad_pcb (KiCad board)
At the start: 2 copper layers, 19 x 19 mm, 8 parts, among them J1 1, J2 2, J3 3, J4 4, J5 5, J6 6

Commit message: completed high density X templates, updated versionnumbers of high density XN templates
Parts:
- N1: value V20220113 -> V20240506
Changed lines of the file:
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@@
   )
   (net 0 "")
-  (net 1 "Net-(J1-Pad1)")
+  (net 1 "Net-(J1-Pin_1)")
   (footprint "mill-max:PC_pin_nail_head_6092" locked (layer "F.Cu")
     (at 142.5 62.5)
+    (property "Sheetfile" "template_1by2_high_density_XN.kicad_sch")
+    (property "Sheetname" "")
+    (property "ki_description" "Generic connector, single row, 01x01, script generated (kicad-library-utils/schlib/autogen/connector/)")
+    (property "ki_keywords" "connector")
     (attr through_hole)
     (fp_text reference "J1" (at 3 0) (layer "F.Fab")
@@
       (stroke (width 0.025) (type solid)) (fill none) (layer "F.CrtYd"))
     (pad "1" thru_hole circle locked (at 0 0) (size 2 2) (drill 1.1) (layers "*.Cu" "*.Mask")
-      (net 1 "Net-(J1-Pad1)"))
+      (net 1 "Net-(J1-Pin_1)") (pinfunction "Pin_1") (pintype "passive"))
   )
   (footprint "mill-max:PC_pin_nail_head_6092" locked (layer "F.Cu")
     (at 142.5 70)
+    (property "Sheetfile" "template_1by2_high_density_XN.kicad_sch")
+    (property "Sheetname" "")
+    (property "ki_description" "Generic connector, single row, 01x01, script generated (kicad-library-utils/schlib/autogen/connector/)")
+    (property "ki_keywords" "connector")
     (attr through_hole)
     (fp_text reference "J2" (at 3 0) (layer "F.Fab")
@@
       (stroke (width 0.025) (type solid)) (fill none) (layer "F.CrtYd"))
     (pad "1" thru_hole circle locked (at 0 0) (size 2 2) (drill 1.1) (layers "*.Cu" "*.Mask")
-      (net 1 "Net-(J1-Pad1)"))
+      (net 1 "Net-(J1-Pin_1)") (pinfunction "Pin_1") (pintype "passive"))
   )
   (footprint "mill-max:PC_pin_nail_head_6092" locked (layer "F.Cu")
     (at 142.5 77.5)
+    (property "Sheetfile" "template_1by2_high_density_XN.kicad_sch")
+    (property "Sheetname" "")
+    (property "ki_description" "Generic connector, single row, 01x01, script generated (kicad-library-utils/schlib/autogen/connector/)")
+    (property "ki_keywords" "connector")
     (attr through_hole)
     (fp_text reference "J3" (at 3 0) (layer "F.Fab")
@@
       (stroke (width 0.025) (type solid)) (fill none) (layer "F.CrtYd"))
     (pad "1" thru_hole circle locked (at 0 0) (size 2 2) (drill 1.1) (layers "*.Cu" "*.Mask")
-      (net 1 "Net-(J1-Pad1)"))
+      (net 1 "Net-(J1-Pin_1)") (pinfunction "Pin_1") (pintype "passive"))
   )
   (footprint "mill-max:PC_pin_nail_head_6092" locked (layer "F.Cu")
     (at 157.5 70)
+    (property "Sheetfile" "template_1by2_high_density_XN.kicad_sch")
+    (property "Sheetname" "")
+    (property "ki_description" "Generic connector, single row, 01x01, script generated (kicad-library-utils/schlib/autogen/connector/)")
+    (property "ki_keywords" "connector")
     (attr through_hole)
     (fp_text reference "J5" (at -3 0) (layer "F.Fab")
@@
       (stroke (width 0.025) (type solid)) (fill none) (layer "F.CrtYd"))
     (pad "1" thru_hole circle locked (at 0 0) (size 2 2) (drill 1.1) (layers "*.Cu" "*.Mask")
-      (net 1 "Net-(J1-Pad1)"))
+      (net 1 "Net-(J1-Pin_1)") (pinfunction "Pin_1") (pintype "passive"))
   )
   (footprint "mill-max:PC_pin_nail_head_6092" locked (layer "F.Cu")
     (at 157.5 62.5)
+    (property "Sheetfile" "template_1by2_high_density_XN.kicad_sch")
+    (property "Sheetname" "")
+    (property "ki_description" "Generic connector, single row, 01x01, script generated (kicad-library-utils/schlib/autogen/connector/)")
+    (property "ki_keywords" "connector")
     (attr through_hole)
     (fp_text reference "J6" (at -3 0) (layer "F.Fab")
@@
       (stroke (width 0.025) (type solid)) (fill none) (layer "F.CrtYd"))
     (pad "1" thru_hole circle locked (at 0 0) (size 2 2) (drill 1.1) (layers "*.Cu" "*.Mask")
-      (net 1 "Net-(J1-Pad1)"))
+      (net 1 "Net-(J1-Pin_1)") (pinfunction "Pin_1") (pintype "passive"))
   )
   (footprint "mill-max:PC_pin_nail_head_6092" locked (layer "F.Cu")
     (at 157.5 77.5)
+    (property "Sheetfile" "template_1by2_high_density_XN.kicad_sch")
+    (property "Sheetname" "")
+    (property "ki_description" "Generic connector, single row, 01x01, script generated (kicad-library-utils/schlib/autogen/connector/)")
+    (property "ki_keywords" "connector")
     (attr through_hole)
     (fp_text reference "J4" (at -3 0) (layer "F.Fab")
@@
       (stroke (width 0.025) (type solid)) (fill none) (layer "F.CrtYd"))
     (pad "1" thru_hole circle locked (at 0 0) (size 2 2) (drill 1.1) (layers "*.Cu" "*.Mask")
-      (net 1 "Net-(J1-Pad1)"))
+      (net 1 "Net-(J1-Pin_1)") (pinfunction "Pin_1") (pintype "passive"))
   )
   (footprint "Symbol:OSHW-Symbol_6.7x6mm_SilkScreen" (layer "B.Cu")
@@
     (descr "Open Source Hardware Symbol")
     (tags "Logo Symbol OSHW")
-    (attr exclude_from_pos_files exclude_from_bom)
+    (property "Sheetfile" "template_1by2_high_density_XN.kicad_sch")
+    (property "Sheetname" "")
+    (attr exclude_from_pos_files)
     (fp_text reference "N2" (at 0 0) (layer "B.SilkS") hide
         (effects (font (size 1 1) (thickness 0.15)) (justify mirror))
@@
     (descr "Label for general purpose use")
     (tags "Label")
+    (property "Sheetfile" "template_1by2_high_density_XN.kicad_sch")
+    (property "Sheetname" "")
     (attr smd)
     (fp_text reference "N1" (at 0 -1.85) (layer "B.Fab") hide
         (effects (font (size 1 1) (thickness 0.15)) (justify mirror))
     )
-    (fp_text value "V20220113" (at 0.8 0.1) (layer "B.SilkS")
+    (fp_text value "V20240506" (at 0.8 0.1) (layer "B.SilkS")
         (effects (font (size 0.8 0.8) (thickness 0.15)) (justify mirror))
     )
