File: electronics/template_1by4_high_density_XN/template_1by4_high_density_XN.kicad_pcb (KiCad board)
At the start: 2 copper layers, 19 x 34 mm, 12 parts, among them J1 1, J10 10, J2 2, J3 3, J4 4, J5 5, J6 6, J7 7, J8 8, J9 9

Commit message: completed high density X templates, updated versionnumbers of high density XN templates
Parts:
- N1: value V20220113 -> V20240506
Changed lines of the file:
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@@
   (footprint "mill-max:PC_pin_nail_head_6092" locked (layer "F.Cu")
     (at 142.5 62.5)
-    (property "Sheetfile" "template_1by4.kicad_sch")
+    (property "Sheetfile" "template_1by4_high_density_XN.kicad_sch")
     (property "Sheetname" "")
     (property "ki_description" "Generic connector, single row, 01x01, script generated (kicad-library-utils/schlib/autogen/connector/)")
@@
   (footprint "mill-max:PC_pin_nail_head_6092" locked (layer "F.Cu")
     (at 142.5 70)
-    (property "Sheetfile" "template_1by4.kicad_sch")
+    (property "Sheetfile" "template_1by4_high_density_XN.kicad_sch")
     (property "Sheetname" "")
     (property "ki_description" "Generic connector, single row, 01x01, script generated (kicad-library-utils/schlib/autogen/connector/)")
@@
   (footprint "mill-max:PC_pin_nail_head_6092" locked (layer "F.Cu")
     (at 142.5 77.5)
-    (property "Sheetfile" "template_1by4.kicad_sch")
+    (property "Sheetfile" "template_1by4_high_density_XN.kicad_sch")
     (property "Sheetname" "")
     (property "ki_description" "Generic connector, single row, 01x01, script generated (kicad-library-utils/schlib/autogen/connector/)")
@@
   (footprint "mill-max:PC_pin_nail_head_6092" locked (layer "F.Cu")
     (at 142.5 92.5 180)
-    (property "Sheetfile" "template_1by4.kicad_sch")
+    (property "Sheetfile" "template_1by4_high_density_XN.kicad_sch")
     (property "Sheetname" "")
     (property "ki_description" "Generic connector, single row, 01x01, script generated (kicad-library-utils/schlib/autogen/connector/)")
@@
   (footprint "mill-max:PC_pin_nail_head_6092" locked (layer "F.Cu")
     (at 157.5 92.5)
-    (property "Sheetfile" "template_1by4.kicad_sch")
+    (property "Sheetfile" "template_1by4_high_density_XN.kicad_sch")
     (property "Sheetname" "")
     (property "ki_description" "Generic connector, single row, 01x01, script generated (kicad-library-utils/schlib/autogen/connector/)")
@@
   (footprint "mill-max:PC_pin_nail_head_6092" locked (layer "F.Cu")
     (at 142.5 85 180)
-    (property "Sheetfile" "template_1by4.kicad_sch")
+    (property "Sheetfile" "template_1by4_high_density_XN.kicad_sch")
     (property "Sheetname" "")
     (property "ki_description" "Generic connector, single row, 01x01, script generated (kicad-library-utils/schlib/autogen/connector/)")
@@
   (footprint "mill-max:PC_pin_nail_head_6092" locked (layer "F.Cu")
     (at 157.5 77.5)
-    (property "Sheetfile" "template_1by4.kicad_sch")
+    (property "Sheetfile" "template_1by4_high_density_XN.kicad_sch")
     (property "Sheetname" "")
     (property "ki_description" "Generic connector, single row, 01x01, script generated (kicad-library-utils/schlib/autogen/connector/)")
@@
   (footprint "mill-max:PC_pin_nail_head_6092" locked (layer "F.Cu")
     (at 157.5 62.5)
-    (property "Sheetfile" "template_1by4.kicad_sch")
+    (property "Sheetfile" "template_1by4_high_density_XN.kicad_sch")
     (property "Sheetname" "")
     (property "ki_description" "Generic connector, single row, 01x01, script generated (kicad-library-utils/schlib/autogen/connector/)")
@@
   (footprint "mill-max:PC_pin_nail_head_6092" locked (layer "F.Cu")
     (at 157.5 85)
-    (property "Sheetfile" "template_1by4.kicad_sch")
+    (property "Sheetfile" "template_1by4_high_density_XN.kicad_sch")
     (property "Sheetname" "")
     (property "ki_description" "Generic connector, single row, 01x01, script generated (kicad-library-utils/schlib/autogen/connector/)")
@@
   (footprint "mill-max:PC_pin_nail_head_6092" locked (layer "F.Cu")
     (at 157.5 70)
-    (property "Sheetfile" "template_1by4.kicad_sch")
+    (property "Sheetfile" "template_1by4_high_density_XN.kicad_sch")
     (property "Sheetname" "")
     (property "ki_description" "Generic connector, single row, 01x01, script generated (kicad-library-utils/schlib/autogen/connector/)")
@@
     (descr "Open Source Hardware Symbol")
     (tags "Logo Symbol OSHW")
-    (property "Sheetfile" "template_1by4.kicad_sch")
+    (property "Sheetfile" "template_1by4_high_density_XN.kicad_sch")
     (property "Sheetname" "")
     (attr exclude_from_pos_files)
@@
     (descr "Label for general purpose use")
     (tags "Label")
-    (property "Sheetfile" "template_1by4.kicad_sch")
+    (property "Sheetfile" "template_1by4_high_density_XN.kicad_sch")
     (property "Sheetname" "")
     (attr smd)
@@
         (effects (font (size 1 1) (thickness 0.15)) (justify mirror))
     )
-    (fp_text value "V20220113" (at 0.8 0.1) (layer "B.SilkS")
+    (fp_text value "V20240506" (at 0.8 0.1) (layer "B.SilkS")
         (effects (font (size 0.8 0.8) (thickness 0.15)) (justify mirror))
     )
