File: electronics/template_1by1/template_1by1.kicad_pcb (KiCad board)
At the start: 2 copper layers, 19 x 19 mm, 6 parts, among them J1 LEFT_TOP, J2 LEFT_BOT, J3 RIGHT_TOP, J4 RIGHT_BOT

Commit message: updated 1 by 1 template
Parts:
- J1: value LEFT_TOP -> 1
- J2: value LEFT_BOT -> 2
- J3: value RIGHT_TOP -> 4
- J4: value RIGHT_BOT -> 3
- N1: value 20201118 -> 20201120
Changed lines of the file:
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@@
   (module mill-max:PC_pin_nail_head_6092 locked (layer F.Cu)
     (at 157 78)
-    (fp_text reference J4 (at -3 0) (layer F.Fab)
+    (fp_text reference J4 (at -2 -2) (layer F.Fab)
       (effects (font (size 1 1) (thickness 0.15)))
     )
-    (fp_text value RIGHT_BOT (at -3 -3) (layer F.SilkS)
+    (fp_text value 3 (at -2 -2) (layer F.SilkS)
       (effects (font (size 1 1) (thickness 0.15)))
     )
+    (fp_circle (center 0 0) (end 1.3 0) (layer B.CrtYd) (width 0.025))
     (fp_circle (center 0 0) (end 1.3 0) (layer F.CrtYd) (width 0.025))
-    (fp_circle (center 0 0) (end 1.3 0) (layer B.CrtYd) (width 0.025))
     (pad 1 thru_hole circle (at 0 0) (size 2 2) (drill 1.1) (layers *.Cu *.Mask)
       (net 1 "Net-(J1-Pad1)"))
@@
   (module mill-max:PC_pin_nail_head_6092 locked (layer F.Cu)
     (at 157 63)
-    (fp_text reference J3 (at -3 0) (layer F.Fab)
+    (fp_text reference J3 (at -2 2) (layer F.Fab)
       (effects (font (size 1 1) (thickness 0.15)))
     )
-    (fp_text value RIGHT_TOP (at -3 3) (layer F.SilkS)
+    (fp_text value 4 (at -2 2) (layer F.SilkS)
       (effects (font (size 1 1) (thickness 0.15)))
     )
+    (fp_circle (center 0 0) (end 1.3 0) (layer B.CrtYd) (width 0.025))
     (fp_circle (center 0 0) (end 1.3 0) (layer F.CrtYd) (width 0.025))
-    (fp_circle (center 0 0) (end 1.3 0) (layer B.CrtYd) (width 0.025))
     (pad 1 thru_hole circle (at 0 0) (size 2 2) (drill 1.1) (layers *.Cu *.Mask)
       (net 1 "Net-(J1-Pad1)"))
@@
   (module mill-max:PC_pin_nail_head_6092 locked (layer F.Cu)
     (at 142 78)
-    (fp_text reference J2 (at 3 0) (layer F.Fab)
+    (fp_text reference J2 (at 2 -2) (layer F.Fab)
       (effects (font (size 1 1) (thickness 0.15)))
     )
-    (fp_text value LEFT_BOT (at 3 -3) (layer F.SilkS)
+    (fp_text value 2 (at 2 -2) (layer F.SilkS)
       (effects (font (size 1 1) (thickness 0.15)))
     )
+    (fp_circle (center 0 0) (end 1.3 0) (layer B.CrtYd) (width 0.025))
     (fp_circle (center 0 0) (end 1.3 0) (layer F.CrtYd) (width 0.025))
-    (fp_circle (center 0 0) (end 1.3 0) (layer B.CrtYd) (width 0.025))
     (pad 1 thru_hole circle (at 0 0) (size 2 2) (drill 1.1) (layers *.Cu *.Mask)
       (net 1 "Net-(J1-Pad1)"))
@@
   (module mill-max:PC_pin_nail_head_6092 locked (layer F.Cu)
     (at 142 63)
-    (fp_text reference J1 (at 3 0) (layer F.Fab)
+    (fp_text reference J1 (at 2 2) (layer F.Fab)
       (effects (font (size 1 1) (thickness 0.15)))
     )
-    (fp_text value LEFT_TOP (at 3 3) (layer F.SilkS)
+    (fp_text value 1 (at 2 2) (layer F.SilkS)
       (effects (font (size 1 1) (thickness 0.15)))
     )
+    (fp_circle (center 0 0) (end 1.3 0) (layer B.CrtYd) (width 0.025))
     (fp_circle (center 0 0) (end 1.3 0) (layer F.CrtYd) (width 0.025))
-    (fp_circle (center 0 0) (end 1.3 0) (layer B.CrtYd) (width 0.025))
     (pad 1 thru_hole circle (at 0 0) (size 2 2) (drill 1.1) (layers *.Cu *.Mask)
       (net 1 "Net-(J1-Pad1)"))
@@
       (effects (font (size 1 1) (thickness 0.15)) (justify mirror))
     )
-    (fp_text value 20201118 (at 0.8 0.1) (layer B.SilkS)
+    (fp_text value 20201120 (at 0.8 0.1) (layer B.SilkS)
       (effects (font (size 0.8 0.8) (thickness 0.15)) (justify mirror))
     )

Commit message: changed font size on the templates
Parts:
- N1: value 20201120 -> V20220113
Changed lines of the file:
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@@
-(kicad_pcb (version 20171130) (host pcbnew 5.1.8-db9833491~87~ubuntu20.04.1)
+(kicad_pcb (version 20171130) (host pcbnew 5.99.0+really5.1.10+dfsg1-1)
   (general
     (thickness 1.6)
@@
     )
     (fp_text value 3 (at -2 -2) (layer F.SilkS)
-      (effects (font (size 1 1) (thickness 0.15)))
+      (effects (font (size 2 2) (thickness 0.3)))
     )
     (fp_circle (center 0 0) (end 1.3 0) (layer B.CrtYd) (width 0.025))
@@
     )
     (fp_text value 4 (at -2 2) (layer F.SilkS)
-      (effects (font (size 1 1) (thickness 0.15)))
+      (effects (font (size 2 2) (thickness 0.3)))
     )
     (fp_circle (center 0 0) (end 1.3 0) (layer B.CrtYd) (width 0.025))
@@
     )
     (fp_text value 2 (at 2 -2) (layer F.SilkS)
-      (effects (font (size 1 1) (thickness 0.15)))
+      (effects (font (size 2 2) (thickness 0.3)))
     )
     (fp_circle (center 0 0) (end 1.3 0) (layer B.CrtYd) (width 0.025))
@@
     )
     (fp_text value 1 (at 2 2) (layer F.SilkS)
-      (effects (font (size 1 1) (thickness 0.15)))
+      (effects (font (size 2 2) (thickness 0.3)))
     )
     (fp_circle (center 0 0) (end 1.3 0) (layer B.CrtYd) (width 0.025))
@@
       (effects (font (size 1 1) (thickness 0.15)) (justify mirror))
     )
-    (fp_text value 20201120 (at 0.8 0.1) (layer B.SilkS)
+    (fp_text value V20220113 (at 0.8 0.1) (layer B.SilkS)
       (effects (font (size 0.8 0.8) (thickness 0.15)) (justify mirror))
     )

Commit message: updated 1 by 1 template
Other:
- net class Default removed
- rule pad_to_mask_clearance: 0.0762 -> 0
