File: electronics/template_1by2/template_1by2.kicad_pcb (KiCad board)
At the start: 2 copper layers, 19 x 34 mm, 8 parts, among them J1 1, J2 2, J3 3, J4 4, J5 5, J6 6

Commit message: locked pins and updated versionnumber
Parts:
- N1: value 20201119 -> 20201120
Changed lines of the file:
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@@
     (add_net "Net-(J1-Pad1)")
   )
-  (module mill-max:PC_pin_nail_head_6092 (layer F.Cu)
+  (module mill-max:PC_pin_nail_head_6092 locked (layer F.Cu)
     (at 157 63)
     (fp_text reference J6 (at -2 2) (layer F.Fab)
@@
       (effects (font (size 1 1) (thickness 0.15)))
     )
+    (fp_circle (center 0 0) (end 1.3 0) (layer B.CrtYd) (width 0.025))
     (fp_circle (center 0 0) (end 1.3 0) (layer F.CrtYd) (width 0.025))
-    (fp_circle (center 0 0) (end 1.3 0) (layer B.CrtYd) (width 0.025))
     (pad 1 thru_hole circle (at 0 0) (size 2 2) (drill 1.1) (layers *.Cu *.Mask)
       (net 1 "Net-(J1-Pad1)"))
   )
-  (module mill-max:PC_pin_nail_head_6092 (layer F.Cu)
+  (module mill-max:PC_pin_nail_head_6092 locked (layer F.Cu)
     (at 157 78)
     (fp_text reference J5 (at -3 0) (layer F.Fab)
@@
       (effects (font (size 1 1) (thickness 0.15)))
     )
+    (fp_circle (center 0 0) (end 1.3 0) (layer B.CrtYd) (width 0.025))
     (fp_circle (center 0 0) (end 1.3 0) (layer F.CrtYd) (width 0.025))
-    (fp_circle (center 0 0) (end 1.3 0) (layer B.CrtYd) (width 0.025))
     (pad 1 thru_hole circle (at 0 0) (size 2 2) (drill 1.1) (layers *.Cu *.Mask)
       (net 1 "Net-(J1-Pad1)"))
@@
       (effects (font (size 1 1) (thickness 0.15)))
     )
+    (fp_circle (center 0 0) (end 1.3 0) (layer F.CrtYd) (width 0.025))
     (fp_circle (center 0 0) (end 1.3 0) (layer B.CrtYd) (width 0.025))
-    (fp_circle (center 0 0) (end 1.3 0) (layer F.CrtYd) (width 0.025))
     (pad 1 thru_hole circle (at 0 0) (size 2 2) (drill 1.1) (layers *.Cu *.Mask)
       (net 1 "Net-(J1-Pad1)"))
@@
       (effects (font (size 1 1) (thickness 0.15)))
     )
+    (fp_circle (center 0 0) (end 1.3 0) (layer F.CrtYd) (width 0.025))
     (fp_circle (center 0 0) (end 1.3 0) (layer B.CrtYd) (width 0.025))
-    (fp_circle (center 0 0) (end 1.3 0) (layer F.CrtYd) (width 0.025))
     (pad 1 thru_hole circle (at 0 0) (size 2 2) (drill 1.1) (layers *.Cu *.Mask)
       (net 1 "Net-(J1-Pad1)"))
@@
       (effects (font (size 1 1) (thickness 0.15)))
     )
+    (fp_circle (center 0 0) (end 1.3 0) (layer F.CrtYd) (width 0.025))
     (fp_circle (center 0 0) (end 1.3 0) (layer B.CrtYd) (width 0.025))
-    (fp_circle (center 0 0) (end 1.3 0) (layer F.CrtYd) (width 0.025))
     (pad 1 thru_hole circle (at 0 0) (size 2 2) (drill 1.1) (layers *.Cu *.Mask)
       (net 1 "Net-(J1-Pad1)"))
@@
       (effects (font (size 1 1) (thickness 0.15)))
     )
+    (fp_circle (center 0 0) (end 1.3 0) (layer F.CrtYd) (width 0.025))
     (fp_circle (center 0 0) (end 1.3 0) (layer B.CrtYd) (width 0.025))
-    (fp_circle (center 0 0) (end 1.3 0) (layer F.CrtYd) (width 0.025))
     (pad 1 thru_hole circle (at 0 0) (size 2 2) (drill 1.1) (layers *.Cu *.Mask)
       (net 1 "Net-(J1-Pad1)"))
@@
       (effects (font (size 1 1) (thickness 0.15)) (justify mirror))
     )
-    (fp_text value 20201119 (at 0.8 0.1) (layer B.SilkS)
+    (fp_text value 20201120 (at 0.8 0.1) (layer B.SilkS)
       (effects (font (size 0.8 0.8) (thickness 0.15)) (justify mirror))
     )

Commit message: changed font size on the templates
Parts:
- N1: value 20201120 -> V20220113
Changed lines of the file:
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@@
-(kicad_pcb (version 20171130) (host pcbnew 5.1.8-db9833491~87~ubuntu20.04.1)
+(kicad_pcb (version 20171130) (host pcbnew 5.99.0+really5.1.10+dfsg1-1)
   (general
     (thickness 1.6)
@@
     )
     (fp_text value 6 (at -2 2) (layer F.SilkS)
-      (effects (font (size 1 1) (thickness 0.15)))
+      (effects (font (size 2 2) (thickness 0.3)))
     )
     (fp_circle (center 0 0) (end 1.3 0) (layer B.CrtYd) (width 0.025))
@@
     )
     (fp_text value 5 (at -3 0) (layer F.SilkS)
-      (effects (font (size 1 1) (thickness 0.15)))
+      (effects (font (size 2 2) (thickness 0.3)))
     )
     (fp_circle (center 0 0) (end 1.3 0) (layer B.CrtYd) (width 0.025))
@@
     )
     (fp_text value 4 (at -2 -2) (layer F.SilkS)
-      (effects (font (size 1 1) (thickness 0.15)))
+      (effects (font (size 2 2) (thickness 0.3)))
     )
     (fp_circle (center 0 0) (end 1.3 0) (layer F.CrtYd) (width 0.025))
@@
     )
     (fp_text value 3 (at 2 -2) (layer F.SilkS)
-      (effects (font (size 1 1) (thickness 0.15)))
+      (effects (font (size 2 2) (thickness 0.3)))
     )
     (fp_circle (center 0 0) (end 1.3 0) (layer F.CrtYd) (width 0.025))
@@
     )
     (fp_text value 2 (at 3 0) (layer F.SilkS)
-      (effects (font (size 1 1) (thickness 0.15)))
+      (effects (font (size 2 2) (thickness 0.3)))
     )
     (fp_circle (center 0 0) (end 1.3 0) (layer F.CrtYd) (width 0.025))
@@
     )
     (fp_text value 1 (at 2 2) (layer F.SilkS)
-      (effects (font (size 1 1) (thickness 0.15)))
+      (effects (font (size 2 2) (thickness 0.3)))
     )
     (fp_circle (center 0 0) (end 1.3 0) (layer F.CrtYd) (width 0.025))
@@
       (effects (font (size 1 1) (thickness 0.15)) (justify mirror))
     )
-    (fp_text value 20201120 (at 0.8 0.1) (layer B.SilkS)
+    (fp_text value V20220113 (at 0.8 0.1) (layer B.SilkS)
       (effects (font (size 0.8 0.8) (thickness 0.15)) (justify mirror))
     )

Commit message: converted to kicad 7
Other:
- net class Default removed
- rule pad_to_mask_clearance: 0.0762 -> 0
