File: electronics/dual_NBJT_mirror_normal/dual_NBJT_mirror_normal.kicad_pcb (KiCad board)
At the start: 2 copper layers, 19 x 34 mm, 8 parts, among them J1 1, J2 2, J3 3, J4 4, J5 5, J6 6

Commit message: SOT363 dual NBJT mirror transistor
Parts:
- added Q1: ~, SquantorIC:SOT363-NXP-hand, F.Cu at (149.5, 78.0)
- J1: value 1 -> C1
- J2: value 2 -> B1
- J3: value 3 -> E1
- J4: value 4 -> E2
- J5: value 5 -> B2
- J6: value 6 -> C2
- N1: value V20220113 -> V20240523
- moved N2 12.0 mm to (149.0, 90.0)
- moved N1 11.5 mm to (148.5, 93.5)
Connections:
- J1 pad 1: Net-(J1-Pad1) -> Net-(J1-Pin_1)
- J2 pad 1: Net-(J1-Pad1) -> Net-(J2-Pin_1)
- J3 pad 1: Net-(J1-Pad1) -> Net-(J3-Pin_1)
- J4 pad 1: Net-(J1-Pad1) -> Net-(J4-Pin_1)
- J5 pad 1: Net-(J1-Pad1) -> Net-(J5-Pin_1)
- J6 pad 1: Net-(J1-Pad1) -> Net-(J6-Pin_1)
Routing:
- net Net-(J6-Pin_1): track 0.00 -> 26.5 mm, vias 0 -> 1
- net Net-(J4-Pin_1): track 0.00 -> 24.6 mm, vias 0 -> 1
- net Net-(J3-Pin_1): track 0.00 -> 22.4 mm, vias 0 -> 1
- net Net-(J1-Pin_1): track 0.00 -> 19.0 mm, vias 0 -> 1
- net Net-(J5-Pin_1): track 0.00 -> 6.45 mm
- net Net-(J2-Pin_1): track 0.00 -> 6.45 mm
