File: electronics/dual_BJT_mirror_XN/dual_BJT_mirror_XN.kicad_pcb (KiCad board)
At the start: 2 copper layers, 19 x 19 mm, 9 parts, among them J1 C1, J2 B1, J3 E1, J4 E2, J5 B2, J6 C2

Commit message: small fixes
Parts:
- moved N1 5.80 mm to (150.9, 78.5)
- moved N2 5.80 mm to (150.0, 74.8)
Routing:
- net Net-(J4-Pin_1): track 10.3 -> 12.4 mm
- net Net-(J6-Pin_1): track 17.6 -> 16.1 mm
- net Net-(J1-Pin_1): track 14.2 -> 15.6 mm
- net Net-(J5-Pin_1): vias 0 -> 1
- net Net-(J2-Pin_1): vias 0 -> 1
Other:
- board text added: "mirrored pinout"
Changed lines of the file:
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@@
   )
   (footprint "Symbol:OSHW-Symbol_6.7x6mm_SilkScreen" (layer "B.Cu")
-    (at 150 69 180)
+    (at 150 74.8 180)
     (descr "Open Source Hardware Symbol")
     (tags "Logo Symbol OSHW")
@@
   )
   (footprint "SquantorLabels:Label_Generic" (layer "B.Cu")
-    (at 150.9 72.7 180)
+    (at 150.9 78.5 180)
     (descr "Label for general purpose use")
     (tags "Label")
@@
   (gr_line (start 140.5 79.5) (end 140.5 60.5)
     (stroke (width 0.05) (type solid)) (layer "Edge.Cuts"))
+  (gr_text "mirrored pinout" (at 150 71) (layer "B.SilkS")
+    (effects (font (size 0.8 0.8) (thickness 0.15) bold) (justify mirror))
+  )
+  (segment (start 151.05 69.25) (end 151.05 68.45) (width 0.4) (layer "F.Cu") (net 1))
   (segment (start 151.05 68.45) (end 151.5 68) (width 0.4) (layer "F.Cu") (net 1))
-  (segment (start 151.05 69.25) (end 151.05 68.45) (width 0.4) (layer "F.Cu") (net 1))
   (via (at 151.5 68) (size 0.8) (drill 0.4) (layers "F.Cu" "B.Cu") (net 1))
-  (segment (start 151.5 68) (end 151.5 65.5) (width 0.4) (layer "B.Cu") (net 1))
-  (segment (start 151.5 65.5) (end 148.5 62.5) (width 0.4) (layer "B.Cu") (net 1))
-  (segment (start 148.5 62.5) (end 142.5 62.5) (width 0.4) (layer "B.Cu") (net 1))
-  (segment (start 148.95 70) (end 142.5 70) (width 0.4) (layer "F.Cu") (net 2))
+  (segment (start 142.5 62.5) (end 151 62.5) (width 0.8) (layer "B.Cu") (net 1))
+  (segment (start 151.5 63) (end 151.5 68) (width 0.8) (layer "B.Cu") (net 1))
+  (segment (start 151 62.5) (end 151.5 63) (width 0.8) (layer "B.Cu") (net 1))
+  (segment (start 148.95 70) (end 147.5 70) (width 0.4) (layer "F.Cu") (net 2))
+  (via (at 147.5 70) (size 0.8) (drill 0.4) (layers "F.Cu" "B.Cu") (net 2))
+  (segment (start 142.5 70) (end 147.5 70) (width 0.8) (layer "B.Cu") (net 2))
+  (segment (start 148.95 69.25) (end 148.95 68.45) (width 0.4) (layer "F.Cu") (net 3))
   (segment (start 148.95 68.45) (end 148.5 68) (width 0.4) (layer "F.Cu") (net 3))
-  (segment (start 148.95 69.25) (end 148.95 68.45) (width 0.4) (layer "F.Cu") (net 3))
   (via (at 148.5 68) (size 0.8) (drill 0.4) (layers "F.Cu" "B.Cu") (net 3))
-  (segment (start 147.5 74) (end 144 77.5) (width 0.4) (layer "B.Cu") (net 3))
-  (segment (start 147.5 68.5) (end 147.5 74) (width 0.4) (layer "B.Cu") (net 3))
-  (segment (start 148 68) (end 147.5 68.5) (width 0.4) (layer "B.Cu") (net 3))
-  (segment (start 148.5 68) (end 148 68) (width 0.4) (layer "B.Cu") (net 3))
-  (segment (start 144 77.5) (end 142.5 77.5) (width 0.4) (layer "B.Cu") (net 3))
+  (segment (start 145.5 76.5) (end 145.5 73.5) (width 0.8) (layer "B.Cu") (net 3))
+  (segment (start 148.5 70.5) (end 148.5 68) (width 0.8) (layer "B.Cu") (net 3))
+  (segment (start 145.5 73.5) (end 148.5 70.5) (width 0.8) (layer "B.Cu") (net 3))
+  (segment (start 142.5 77.5) (end 144.5 77.5) (width 0.8) (layer "B.Cu") (net 3))
+  (segment (start 144.5 77.5) (end 145.5 76.5) (width 0.8) (layer "B.Cu") (net 3))
   (segment (start 151.05 71.55) (end 151.5 72) (width 0.4) (layer "F.Cu") (net 4))
   (segment (start 151.05 70.75) (end 151.05 71.55) (width 0.4) (layer "F.Cu") (net 4))
   (via (at 151.5 72) (size 0.8) (drill 0.4) (layers "F.Cu" "B.Cu") (net 4))
-  (segment (start 156 77.5) (end 157.5 77.5) (width 0.4) (layer "B.Cu") (net 4))
-  (segment (start 151.5 72) (end 151.5 73) (width 0.4) (layer "B.Cu") (net 4))
-  (segment (start 151.5 73) (end 156 77.5) (width 0.4) (layer "B.Cu") (net 4))
-  (segment (start 151.05 70) (end 157.5 70) (width 0.4) (layer "F.Cu") (net 5))
+  (segment (start 152.5 77.5) (end 151.5 76.5) (width 0.8) (layer "B.Cu") (net 4))
+  (segment (start 157.5 77.5) (end 152.5 77.5) (width 0.8) (layer "B.Cu") (net 4))
+  (segment (start 151.5 76.5) (end 151.5 72) (width 0.8) (layer "B.Cu") (net 4))
+  (segment (start 151.05 70) (end 152.5 70) (width 0.4) (layer "F.Cu") (net 5))
+  (via (at 152.5 70) (size 0.8) (drill 0.4) (layers "F.Cu" "B.Cu") (net 5))
+  (segment (start 157.5 70) (end 152.5 70) (width 0.8) (layer "B.Cu") (net 5))
+  (segment (start 148.95 70.75) (end 148.95 71.55) (width 0.4) (layer "F.Cu") (net 6))
   (segment (start 148.95 71.55) (end 148.5 72) (width 0.4) (layer "F.Cu") (net 6))
-  (segment (start 148.95 70.75) (end 148.95 71.55) (width 0.4) (layer "F.Cu") (net 6))
   (via (at 148.5 72) (size 0.8) (drill 0.4) (layers "F.Cu" "B.Cu") (net 6))
-  (segment (start 154 64.5) (end 156 62.5) (width 0.4) (layer "B.Cu") (net 6))
-  (segment (start 148.5 72) (end 149.5 71) (width 0.4) (layer "B.Cu") (net 6))
-  (segment (start 153 71) (end 154 70) (width 0.4) (layer "B.Cu") (net 6))
-  (segment (start 156 62.5) (end 157.5 62.5) (width 0.4) (layer "B.Cu") (net 6))
-  (segment (start 154 70) (end 154 64.5) (width 0.4) (layer "B.Cu") (net 6))
-  (segment (start 149.5 71) (end 153 71) (width 0.4) (layer "B.Cu") (net 6))
+  (segment (start 151 70) (end 150.5 70) (width 0.8) (layer "B.Cu") (net 6))
+  (segment (start 150.5 70) (end 148.5 72) (width 0.8) (layer "B.Cu") (net 6))
+  (segment (start 155.5 62.5) (end 153 65) (width 0.8) (layer "B.Cu") (net 6))
+  (segment (start 153 65) (end 153 68) (width 0.8) (layer "B.Cu") (net 6))
+  (segment (start 157.5 62.5) (end 155.5 62.5) (width 0.8) (layer "B.Cu") (net 6))
+  (segment (start 153 68) (end 151 70) (width 0.8) (layer "B.Cu") (net 6))
 )
