File: electronics/dual_BJT_mirror_normal/dual_BJT_mirror_normal.kicad_pcb (KiCad board)
At the start: 2 copper layers, 19 x 34 mm, 9 parts, among them J1 C1, J2 B1, J3 E1, J4 E2, J5 B2, J6 C2

Commit message: small fixes
Routing:
- net Net-(J4-Pin_1): track 24.6 -> 18.1 mm
- net Net-(J6-Pin_1): track 26.5 -> 25.1 mm
- net Net-(J5-Pin_1): vias 0 -> 1
- net Net-(J2-Pin_1): vias 0 -> 1
Other:
- board text added: "mirrored transistor"
Changed lines of the file:
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@@
     (property "ki_description" "Dual NPN transistor that allows for mirroring of the device")
     (attr smd)
-    (fp_text reference "Q1" (at 0 -2) (layer "F.SilkS")
+    (fp_text reference "Q1" (at 0 -2) (layer "F.SilkS") hide
         (effects (font (size 1 1) (thickness 0.15)))
     )
-    (fp_text value "~" (at 0 2) (layer "F.Fab")
+    (fp_text value "~" (at 0 2) (layer "F.Fab") hide
         (effects (font (size 1 1) (thickness 0.15)))
     )
@@
       (stroke (width 0.15) (type solid)) (layer "B.SilkS"))
   )
+  (gr_rect (start 140.5 86) (end 158.5 91)
+    (stroke (width 0.15) (type solid)) (fill solid) (layer "F.SilkS"))
   (gr_line (start 140 95) (end 159 95)
     (stroke (width 0.05) (type solid)) (layer "Edge.Cuts"))
@@
   (gr_line (start 140 95) (end 140 61)
     (stroke (width 0.05) (type solid)) (layer "Edge.Cuts"))
+  (gr_text "mirrored transistor" (at 149 86) (layer "B.SilkS")
+    (effects (font (size 0.8 0.8) (thickness 0.15) bold) (justify mirror))
+  )
   (segment (start 150.55 77.25) (end 150.55 76.45) (width 0.4) (layer "F.Cu") (net 1))
   (segment (start 150.55 76.45) (end 151 76) (width 0.4) (layer "F.Cu") (net 1))
-  (via (at 151 76) (size 0.7) (drill 0.3) (layers "F.Cu" "B.Cu") (net 1))
-  (segment (start 151 76) (end 151 70.5) (width 0.4) (layer "B.Cu") (net 1))
-  (segment (start 143.5 63) (end 142 63) (width 0.4) (layer "B.Cu") (net 1))
-  (segment (start 151 70.5) (end 143.5 63) (width 0.4) (layer "B.Cu") (net 1))
-  (segment (start 148.45 78) (end 142 78) (width 0.4) (layer "F.Cu") (net 2))
+  (via (at 151 76) (size 0.8) (drill 0.4) (layers "F.Cu" "B.Cu") (net 1))
+  (segment (start 142 63) (end 144 63) (width 0.8) (layer "B.Cu") (net 1))
+  (segment (start 151 70) (end 151 76) (width 0.8) (layer "B.Cu") (net 1))
+  (segment (start 144 63) (end 151 70) (width 0.8) (layer "B.Cu") (net 1))
+  (segment (start 148.45 78) (end 147 78) (width 0.4) (layer "F.Cu") (net 2))
+  (via (at 147 78) (size 0.8) (drill 0.4) (layers "F.Cu" "B.Cu") (net 2))
+  (segment (start 142 78) (end 147 78) (width 0.8) (layer "B.Cu") (net 2))
   (segment (start 148.45 77.25) (end 148.45 76.45) (width 0.4) (layer "F.Cu") (net 3))
   (segment (start 148.45 76.45) (end 148 76) (width 0.4) (layer "F.Cu") (net 3))
-  (via (at 148 76) (size 0.7) (drill 0.3) (layers "F.Cu" "B.Cu") (net 3))
-  (segment (start 146 77) (end 146 90.5) (width 0.4) (layer "B.Cu") (net 3))
-  (segment (start 147 76) (end 146 77) (width 0.4) (layer "B.Cu") (net 3))
-  (segment (start 148 76) (end 147 76) (width 0.4) (layer "B.Cu") (net 3))
-  (segment (start 146 90.5) (end 143.5 93) (width 0.4) (layer "B.Cu") (net 3))
-  (segment (start 143.5 93) (end 142 93) (width 0.4) (layer "B.Cu") (net 3))
+  (via (at 148 76) (size 0.8) (drill 0.4) (layers "F.Cu" "B.Cu") (net 3))
+  (segment (start 148 78.5) (end 148 76) (width 0.8) (layer "B.Cu") (net 3))
+  (segment (start 147 79.5) (end 148 78.5) (width 0.8) (layer "B.Cu") (net 3))
+  (segment (start 147 90) (end 147 79.5) (width 0.8) (layer "B.Cu") (net 3))
+  (segment (start 144 93) (end 147 90) (width 0.8) (layer "B.Cu") (net 3))
+  (segment (start 142 93) (end 144 93) (width 0.8) (layer "B.Cu") (net 3))
   (segment (start 150.55 79.55) (end 151 80) (width 0.4) (layer "F.Cu") (net 4))
   (segment (start 150.55 78.75) (end 150.55 79.55) (width 0.4) (layer "F.Cu") (net 4))
-  (via (at 151 80) (size 0.7) (drill 0.3) (layers "F.Cu" "B.Cu") (net 4))
-  (segment (start 147 79.469669) (end 147 84.5) (width 0.4) (layer "B.Cu") (net 4))
-  (segment (start 147 84.5) (end 155.5 93) (width 0.4) (layer "B.Cu") (net 4))
-  (segment (start 151 80) (end 150 79) (width 0.4) (layer "B.Cu") (net 4))
-  (segment (start 147.469669 79) (end 147 79.469669) (width 0.4) (layer "B.Cu") (net 4))
-  (segment (start 150 79) (end 147.469669 79) (width 0.4) (layer "B.Cu") (net 4))
-  (segment (start 155.5 93) (end 157 93) (width 0.4) (layer "B.Cu") (net 4))
-  (segment (start 150.55 78) (end 157 78) (width 0.4) (layer "F.Cu") (net 5))
+  (via (at 151 80) (size 0.8) (drill 0.4) (layers "F.Cu" "B.Cu") (net 4))
+  (segment (start 157 93) (end 155 93) (width 0.8) (layer "B.Cu") (net 4))
+  (segment (start 155 93) (end 151 89) (width 0.8) (layer "B.Cu") (net 4))
+  (segment (start 151 89) (end 151 80) (width 0.8) (layer "B.Cu") (net 4))
+  (segment (start 150.55 78) (end 152 78) (width 0.4) (layer "F.Cu") (net 5))
+  (via (at 152 78) (size 0.8) (drill 0.4) (layers "F.Cu" "B.Cu") (net 5))
+  (segment (start 157 78) (end 152 78) (width 0.8) (layer "B.Cu") (net 5))
+  (segment (start 148.45 79.55) (end 148 80) (width 0.4) (layer "F.Cu") (net 6))
   (segment (start 148.45 78.75) (end 148.45 79.55) (width 0.4) (layer "F.Cu") (net 6))
-  (segment (start 148.45 79.55) (end 148 80) (width 0.4) (layer "F.Cu") (net 6))
-  (via (at 148 80) (size 0.7) (drill 0.3) (layers "F.Cu" "B.Cu") (net 6))
-  (segment (start 149 81) (end 151.5 81) (width 0.4) (layer "B.Cu") (net 6))
-  (segment (start 151.5 81) (end 152 80.5) (width 0.4) (layer "B.Cu") (net 6))
-  (segment (start 152 80.5) (end 152 66.5) (width 0.4) (layer "B.Cu") (net 6))
-  (segment (start 155.5 63) (end 157 63) (width 0.4) (layer "B.Cu") (net 6))
-  (segment (start 152 66.5) (end 155.5 63) (width 0.4) (layer "B.Cu") (net 6))
-  (segment (start 148 80) (end 149 81) (width 0.4) (layer "B.Cu") (net 6))
+  (via (at 148 80) (size 0.8) (drill 0.4) (layers "F.Cu" "B.Cu") (net 6))
+  (segment (start 155 63) (end 152.5 65.5) (width 0.8) (layer "B.Cu") (net 6))
+  (segment (start 149.5 77.5) (end 149.5 79.5) (width 0.8) (layer "B.Cu") (net 6))
+  (segment (start 149 80) (end 148 80) (width 0.8) (layer "B.Cu") (net 6))
+  (segment (start 152.5 76.457107) (end 151.957107 77) (width 0.8) (layer "B.Cu") (net 6))
+  (segment (start 149.5 79.5) (end 149 80) (width 0.8) (layer "B.Cu") (net 6))
+  (segment (start 150 77) (end 149.5 77.5) (width 0.8) (layer "B.Cu") (net 6))
+  (segment (start 151.957107 77) (end 150 77) (width 0.8) (layer "B.Cu") (net 6))
+  (segment (start 157 63) (end 155 63) (width 0.8) (layer "B.Cu") (net 6))
+  (segment (start 152.5 65.5) (end 152.5 76.457107) (width 0.8) (layer "B.Cu") (net 6))
 )
