File: electronics/breakout_SOT363_normal/breakout_SOT363_normal.kicad_pcb (KiCad board)
At the start: 2 copper layers, 19 x 34 mm, 16 parts, among them J1 1, J2 2, J3 3, J4 4, J5 5, J6 6, U1 generic_5pin_sot

Commit message: small changes
Parts:
- moved R1 1.00 mm to (145.0, 75.0)
- moved R2 1.00 mm to (154.0, 75.0)
- moved R3 1.00 mm to (154.0, 81.0)
- moved R4 1.00 mm to (145.0, 81.0)
Changed lines of the file:
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@@
   )
   (footprint "SquantorResistor:R_0805+0603" (layer "F.Cu")
-    (at 145 82 90)
+    (at 145 81 90)
     (descr "Resistor SMD 0805, reflow soldering, Vishay (see dcrcw.pdf)")
     (tags "resistor 0805")
@@
   )
   (footprint "SquantorResistor:R_0805+0603" (layer "F.Cu")
-    (at 154 74 90)
+    (at 154 75 90)
     (descr "Resistor SMD 0805, reflow soldering, Vishay (see dcrcw.pdf)")
     (tags "resistor 0805")
@@
   )
   (footprint "SquantorResistor:R_0805+0603" (layer "F.Cu")
-    (at 154 82 90)
+    (at 154 81 90)
     (descr "Resistor SMD 0805, reflow soldering, Vishay (see dcrcw.pdf)")
     (tags "resistor 0805")
@@
   )
   (footprint "SquantorResistor:R_0805+0603" (layer "F.Cu")
-    (at 145 74 90)
+    (at 145 75 90)
     (descr "Resistor SMD 0805, reflow soldering, Vishay (see dcrcw.pdf)")
     (tags "resistor 0805")
