File: electronics/TL431_TH/TL431_TH.kicad_pcb (KiCad board)
At the start: 2 copper layers, 19 x 19 mm, 7 parts, among them J1 Ref, J2 C, J3 A, J4 C, U1 TL431

Commit message: review changes
Parts:
- N1: value V20240522 -> V20240530
- U1: footprint SquantorIC:TO-92L_Inline -> SquantorIC:TO-92L_Inline_Wide
Routing:
- net Net-(J1-Pin_1): track 12.9 -> 14.4 mm
- net Net-(J3-Pin_1): track 11.1 -> 10.5 mm
Changed lines of the file:
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@@
   (footprint "mill-max:PC_pin_nail_head_6092" locked (layer "F.Cu")
     (at 142 63)
-    (property "Sheetfile" "template_1by1.kicad_sch")
+    (property "Sheetfile" "TL431_TH.kicad_sch")
     (property "Sheetname" "")
     (property "ki_description" "Generic connector, single row, 01x01, script generated (kicad-library-utils/schlib/autogen/connector/)")
@@
   (footprint "mill-max:PC_pin_nail_head_6092" locked (layer "F.Cu")
     (at 142 78)
-    (property "Sheetfile" "template_1by1.kicad_sch")
+    (property "Sheetfile" "TL431_TH.kicad_sch")
     (property "Sheetname" "")
     (property "ki_description" "Generic connector, single row, 01x01, script generated (kicad-library-utils/schlib/autogen/connector/)")
@@
   (footprint "mill-max:PC_pin_nail_head_6092" locked (layer "F.Cu")
     (at 157 63)
-    (property "Sheetfile" "template_1by1.kicad_sch")
+    (property "Sheetfile" "TL431_TH.kicad_sch")
     (property "Sheetname" "")
     (property "ki_description" "Generic connector, single row, 01x01, script generated (kicad-library-utils/schlib/autogen/connector/)")
@@
   (footprint "mill-max:PC_pin_nail_head_6092" locked (layer "F.Cu")
     (at 157 78)
-    (property "Sheetfile" "template_1by1.kicad_sch")
+    (property "Sheetfile" "TL431_TH.kicad_sch")
     (property "Sheetname" "")
     (property "ki_description" "Generic connector, single row, 01x01, script generated (kicad-library-utils/schlib/autogen/connector/)")
@@
       (net 2 "Net-(J2-Pin_1)") (pinfunction "Pin_1") (pintype "passive"))
   )
-  (footprint "SquantorIC:TO-92L_Inline" (layer "F.Cu")
+  (footprint "SquantorIC:TO-92L_Inline_Wide" (layer "F.Cu")
     (at 149.5 70.5 90)
     (descr "TO-92L leads in-line (large body variant of TO-92), also known as TO-226, wide, drill 0.75mm (see https://www.diodes.com/assets/Package-Files/TO92L.pdf and http://www.ti.com/lit/an/snoa059/snoa059.pdf)")
     (tags "TO-92L Inline Wide transistor")
-    (property "Sheetfile" "template_1by1.kicad_sch")
+    (property "Sheetfile" "TL431_TH.kicad_sch")
     (property "Sheetname" "")
     (attr through_hole)
@@
         (effects (font (size 0.8 0.8) (thickness 0.15)))
     )
-    (fp_text value "TL431" (at 0 2.4 90) (layer "F.Fab") hide
+    (fp_text value "TL431" (at 0 2.4 90) (layer "F.Fab")
         (effects (font (size 0.8 0.8) (thickness 0.15)))
     )
-    (fp_line (start -2.02 1.7) (end 1.83 1.7)
+    (fp_line (start -1.94 1.7) (end 1.91 1.7)
       (stroke (width 0.12) (type solid)) (layer "F.SilkS"))
-    (fp_arc (start -2.02 1.7) (mid -0.086552 -2.579449) (end 1.868611 1.690122)
+    (fp_arc (start -2.3564 -1.098807) (mid -1.396979 -2.192817) (end 0 -2.6)
       (stroke (width 0.12) (type solid)) (layer "F.SilkS"))
-    (fp_line (start -2.82 -2.75) (end -2.82 1.85)
+    (fp_arc (start -1.94 1.7) (mid -2.150817 1.423933) (end -2.322631 1.122045)
+      (stroke (width 0.12) (type solid)) (layer "F.SilkS"))
+    (fp_arc (start 0 -2.6) (mid 1.396979 -2.192818) (end 2.3564 -1.098807)
+      (stroke (width 0.12) (type solid)) (layer "F.SilkS"))
+    (fp_arc (start 2.302383 1.112264) (mid 2.126594 1.419753) (end 1.91 1.7)
+      (stroke (width 0.12) (type solid)) (layer "F.SilkS"))
+    (fp_line (start -3.54 -2.75) (end -3.54 1.85)
       (stroke (width 0.05) (type solid)) (layer "F.CrtYd"))
-    (fp_line (start -2.82 -2.75) (end 2.68 -2.75)
+    (fp_line (start -3.54 -2.75) (end 3.56 -2.75)
       (stroke (width 0.05) (type solid)) (layer "F.CrtYd"))
-    (fp_line (start 2.68 1.85) (end -2.82 1.85)
+    (fp_line (start 3.56 1.85) (end -3.54 1.85)
       (stroke (width 0.05) (type solid)) (layer "F.CrtYd"))
-    (fp_line (start 2.68 1.85) (end 2.68 -2.75)
+    (fp_line (start 3.56 1.85) (end 3.56 -2.75)
       (stroke (width 0.05) (type solid)) (layer "F.CrtYd"))
-    (fp_line (start -1.97 1.6) (end 1.78 1.6)
+    (fp_line (start -1.89 1.6) (end 1.86 1.6)
       (stroke (width 0.1) (type solid)) (layer "F.Fab"))
-    (fp_arc (start -1.972818 1.602385) (mid -2.329924 -1.043188) (end -0.08 -2.48)
+    (fp_arc (start -1.892818 1.602385) (mid -2.249924 -1.043188) (end 0 -2.48)
       (stroke (width 0.1) (type solid)) (layer "F.Fab"))
-    (fp_arc (start -0.08 -2.48) (mid 2.167211 -1.049019) (end 1.821103 1.592547)
+    (fp_arc (start 0 -2.48) (mid 2.247211 -1.049019) (end 1.901103 1.592547)
       (stroke (width 0.1) (type solid)) (layer "F.Fab"))
-    (pad "1" thru_hole rect (at -1.27 0 90) (size 1.05 1.5) (drill 0.75) (layers "*.Cu" "*.Mask")
+    (pad "1" thru_hole rect (at -2.54 0 90) (size 1.5 1.5) (drill 0.8) (layers "*.Cu" "*.Mask")
       (net 1 "Net-(J1-Pin_1)") (pinfunction "REF") (pintype "input"))
-    (pad "2" thru_hole oval (at 0 0 90) (size 1.05 1.5) (drill 0.75) (layers "*.Cu" "*.Mask")
+    (pad "2" thru_hole circle (at 0 0 90) (size 1.5 1.5) (drill 0.8) (layers "*.Cu" "*.Mask")
       (net 2 "Net-(J2-Pin_1)") (pinfunction "A") (pintype "power_in"))
-    (pad "3" thru_hole oval (at 1.27 0 90) (size 1.05 1.5) (drill 0.75) (layers "*.Cu" "*.Mask")
+    (pad "3" thru_hole circle (at 2.54 0 90) (size 1.5 1.5) (drill 0.8) (layers "*.Cu" "*.Mask")
       (net 3 "Net-(J3-Pin_1)") (pinfunction "C") (pintype "power_out"))
-    (model "${KICAD6_3DMODEL_DIR}/Package_TO_SOT_THT.3dshapes/TO-92L_Inline.wrl"
-      (offset (xyz -1.27 0 0))
+    (model "${KICAD6_3DMODEL_DIR}/Package_TO_SOT_THT.3dshapes/TO-92L_Inline_Wide.wrl"
+      (offset (xyz -2.45 0 0))
       (scale (xyz 1 1 1))
       (rotate (xyz 0 0 0))
@@
     (descr "Label for general purpose use")
     (tags "Label")
-    (property "Sheetfile" "template_1by1.kicad_sch")
+    (property "Sheetfile" "TL431_TH.kicad_sch")
     (property "Sheetname" "")
     (attr smd)
@@
         (effects (font (size 1 1) (thickness 0.15)) (justify mirror))
     )
-    (fp_text value "V20240522" (at 0.8 0.1 90) (layer "B.SilkS")
+    (fp_text value "V20240530" (at 0.8 0.1 90) (layer "B.SilkS")
         (effects (font (size 0.8 0.8) (thickness 0.15)) (justify mirror))
     )
@@
     (descr "Open Source Hardware Symbol")
     (tags "Logo Symbol OSHW")
-    (property "Sheetfile" "template_1by1.kicad_sch")
+    (property "Sheetfile" "TL431_TH.kicad_sch")
     (property "Sheetname" "")
     (attr exclude_from_pos_files)
@@
   (gr_line (start 140 80) (end 140 61)
     (stroke (width 0.05) (type solid)) (layer "Edge.Cuts"))
-  (segment (start 142 63) (end 142 66) (width 2) (layer "B.Cu") (net 1))
-  (segment (start 149.5 71.77) (end 147.77 71.77) (width 1) (layer "B.Cu") (net 1))
-  (segment (start 142 66) (end 147.5 71.5) (width 2) (layer "B.Cu") (net 1))
-  (segment (start 147.77 71.77) (end 147.5 71.5) (width 1) (layer "B.Cu") (net 1))
+  (segment (start 148.097 73.04) (end 142 66.943) (width 2) (layer "B.Cu") (net 1))
+  (segment (start 149.5 73.04) (end 148.097 73.04) (width 2) (layer "B.Cu") (net 1))
+  (segment (start 149.04 73.04) (end 149.5 73.04) (width 1) (layer "B.Cu") (net 1))
+  (segment (start 142 66.943) (end 142 63) (width 2) (layer "B.Cu") (net 1))
   (segment (start 142 78) (end 153.5 78) (width 2) (layer "B.Cu") (net 2))
+  (segment (start 151.5 70.5) (end 149.5 70.5) (width 2) (layer "B.Cu") (net 2))
   (segment (start 153.5 78) (end 153.5 72.5) (width 2) (layer "B.Cu") (net 2))
   (segment (start 153.5 72.5) (end 151.5 70.5) (width 2) (layer "B.Cu") (net 2))
   (segment (start 153.5 78) (end 157 78) (width 2) (layer "B.Cu") (net 2))
-  (segment (start 149.5 70.5) (end 151.5 70.5) (width 1) (layer "B.Cu") (net 2))
-  (segment (start 157 63) (end 154 63) (width 2) (layer "B.Cu") (net 3))
-  (segment (start 154 63) (end 149.5 67.5) (width 2) (layer "B.Cu") (net 3))
-  (segment (start 149.5 69.23) (end 149.5 67.5) (width 1) (layer "B.Cu") (net 3))
+  (segment (start 152.773 63) (end 149.5 66.273) (width 2) (layer "B.Cu") (net 3))
+  (segment (start 149.5 66.273) (end 149.5 67.96) (width 2) (layer "B.Cu") (net 3))
+  (segment (start 157 63) (end 152.773 63) (width 2) (layer "B.Cu") (net 3))
 )
