File: electronics/dual_opamp_normal/dual_opamp_normal.kicad_pcb (KiCad board)
At the start: 2 copper layers, 19 x 49 mm, 12 parts, among them J1 OUT1, J2 -IN1, J3 +IN1, J4 V-, J5 +IN2, J6 -IN2, J7 OUT2, J8 V+, U1 opamp_dual_8pin

Commit message: updated symbol/footprint tables
Parts:
- C1: footprint SquantorCapacitor:C-050-050X080-film -> SquantorCapacitor:C-050-050X100-0805-3516-film
Changed lines of the file:
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@@
   (footprint "mill-max:PC_pin_nail_head_6092" locked (layer "F.Cu")
     (at 142 63)
-    (property "Sheetfile" "template_1by3.kicad_sch")
+    (property "Sheetfile" "dual_opamp_normal.kicad_sch")
     (property "Sheetname" "")
     (property "ki_description" "Generic connector, single row, 01x01, script generated (kicad-library-utils/schlib/autogen/connector/)")
@@
   (footprint "mill-max:PC_pin_nail_head_6092" locked (layer "F.Cu")
     (at 142 78)
-    (property "Sheetfile" "template_1by3.kicad_sch")
+    (property "Sheetfile" "dual_opamp_normal.kicad_sch")
     (property "Sheetname" "")
     (property "ki_description" "Generic connector, single row, 01x01, script generated (kicad-library-utils/schlib/autogen/connector/)")
@@
   (footprint "mill-max:PC_pin_nail_head_6092" locked (layer "F.Cu")
     (at 142 93)
-    (property "Sheetfile" "template_1by3.kicad_sch")
+    (property "Sheetfile" "dual_opamp_normal.kicad_sch")
     (property "Sheetname" "")
     (property "ki_description" "Generic connector, single row, 01x01, script generated (kicad-library-utils/schlib/autogen/connector/)")
@@
   (footprint "mill-max:PC_pin_nail_head_6092" locked (layer "F.Cu")
     (at 157 108)
-    (property "Sheetfile" "template_1by3.kicad_sch")
+    (property "Sheetfile" "dual_opamp_normal.kicad_sch")
     (property "Sheetname" "")
     (property "ki_description" "Generic connector, single row, 01x01, script generated (kicad-library-utils/schlib/autogen/connector/)")
@@
   (footprint "mill-max:PC_pin_nail_head_6092" locked (layer "F.Cu")
     (at 157 93)
-    (property "Sheetfile" "template_1by3.kicad_sch")
+    (property "Sheetfile" "dual_opamp_normal.kicad_sch")
     (property "Sheetname" "")
     (property "ki_description" "Generic connector, single row, 01x01, script generated (kicad-library-utils/schlib/autogen/connector/)")
@@
   (footprint "mill-max:PC_pin_nail_head_6092" locked (layer "F.Cu")
     (at 142 108)
-    (property "Sheetfile" "template_1by3.kicad_sch")
+    (property "Sheetfile" "dual_opamp_normal.kicad_sch")
     (property "Sheetname" "")
     (property "ki_description" "Generic connector, single row, 01x01, script generated (kicad-library-utils/schlib/autogen/connector/)")
@@
   (footprint "mill-max:PC_pin_nail_head_6092" locked (layer "F.Cu")
     (at 157 78)
-    (property "Sheetfile" "template_1by3.kicad_sch")
+    (property "Sheetfile" "dual_opamp_normal.kicad_sch")
     (property "Sheetname" "")
     (property "ki_description" "Generic connector, single row, 01x01, script generated (kicad-library-utils/schlib/autogen/connector/)")
@@
   (footprint "mill-max:PC_pin_nail_head_6092" locked (layer "F.Cu")
     (at 157 63)
-    (property "Sheetfile" "template_1by3.kicad_sch")
+    (property "Sheetfile" "dual_opamp_normal.kicad_sch")
     (property "Sheetname" "")
     (property "ki_description" "Generic connector, single row, 01x01, script generated (kicad-library-utils/schlib/autogen/connector/)")
@@
       (net 2 "Net-(J8-Pin_1)") (pinfunction "Pin_1") (pintype "passive"))
   )
-  (footprint "SquantorCapacitor:C-050-050X080-film" (layer "F.Cu")
+  (footprint "SquantorCapacitor:C-050-050X100-0805-3516-film" (layer "F.Cu")
     (at 149.5 76)
-    (descr "Through hole Film capacitor pitch 5.0mm size 5.0 by 8.0mm")
-    (tags "Film capacitor")
-    (property "Sheetfile" "template_1by3.kicad_sch")
+    (descr "Through hole Film capacitor with SMT 5.0mm pitch size 5.0 by 10.0mm and 0805 to 2512")
+    (tags "Film capacitor multipitch TH SMT")
+    (property "Sheetfile" "dual_opamp_normal.kicad_sch")
     (property "Sheetname" "")
     (property "ki_description" "Unpolarized capacitor")
     (property "ki_keywords" "cap capacitor")
     (attr through_hole)
-    (fp_text reference "C1" (at 0 -1.75) (layer "F.SilkS")
+    (fp_text reference "C1" (at 0 -3.5) (layer "F.SilkS")
         (effects (font (size 0.8 0.8) (thickness 0.15)))
     )
-    (fp_text value "1u" (at 0 3.6) (layer "F.Fab")
+    (fp_text value "1u" (at 0 3.7) (layer "F.Fab")
         (effects (font (size 0.8 0.8) (thickness 0.15)))
     )
-    (fp_line (start -3.600001 -2.100001) (end -3.600001 2.100001)
-      (stroke (width 0.15) (type solid)) (layer "F.SilkS"))
-    (fp_line (start -3.100001 2.600001) (end 3.1 2.6)
-      (stroke (width 0.15) (type solid)) (layer "F.SilkS"))
-    (fp_line (start -0.3 -1) (end -0.3 1)
-      (stroke (width 0.15) (type default)) (layer "F.SilkS"))
-    (fp_line (start -0.3 0) (end -1.3 0)
-      (stroke (width 0.15) (type default)) (layer "F.SilkS"))
-    (fp_line (start 0.3 -1) (end 0.3 1)
-      (stroke (width 0.15) (type default)) (layer "F.SilkS"))
-    (fp_line (start 0.3 0) (end 1.3 0)
-      (stroke (width 0.15) (type default)) (layer "F.SilkS"))
-    (fp_line (start 3.1 -2.6) (end -3.100001 -2.600001)
-      (stroke (width 0.15) (type solid)) (layer "F.SilkS"))
-    (fp_line (start 3.6 2.1) (end 3.6 -2)
-      (stroke (width 0.15) (type solid)) (layer "F.SilkS"))
-    (fp_arc (start -3.600001 -2.100001) (mid -3.453554 -2.453554) (end -3.100001 -2.600001)
-      (stroke (width 0.15) (type solid)) (layer "F.SilkS"))
-    (fp_arc (start -3.100001 2.600001) (mid -3.453554 2.453554) (end -3.600001 2.100001)
-      (stroke (width 0.15) (type solid)) (layer "F.SilkS"))
-    (fp_arc (start 3.1 -2.6) (mid 3.453553 -2.453553) (end 3.6 -2.1)
-      (stroke (width 0.15) (type solid)) (layer "F.SilkS"))
-    (fp_arc (start 3.6 2.1) (mid 3.453553 2.453553) (end 3.1 2.6)
-      (stroke (width 0.15) (type solid)) (layer "F.SilkS"))
-    (fp_line (start -4 -3) (end -4 3)
+    (fp_text user "${REFERENCE}" (at 0 -3.5) (layer "B.SilkS")
+        (effects (font (size 0.8 0.8) (thickness 0.15)) (justify mirror))
+    )
+    (fp_text user "${VALUE}" (at 0 3.7) (layer "B.Fab")
+        (effects (font (size 0.8 0.8) (thickness 0.15)) (justify mirror))
+    )
+    (fp_line (start 0 -2) (end 0 -0.5)
+      (stroke (width 0.15) (type solid)) (layer "B.SilkS"))
+    (fp_line (start 0 2) (end 0 0.5)
+      (stroke (width 0.15) (type solid)) (layer "B.SilkS"))
+    (fp_line (start -3.75 -2) (end -3.75 2)
+      (stroke (width 0.15) (type solid)) (layer "F.SilkS"))
+    (fp_line (start -3.25 2.5) (end 3.25 2.5)
+      (stroke (width 0.15) (type solid)) (layer "F.SilkS"))
+    (fp_line (start 3.25 -2.5) (end -3.25 -2.5)
+      (stroke (width 0.15) (type solid)) (layer "F.SilkS"))
+    (fp_line (start 3.75 2) (end 3.75 -2)
+      (stroke (width 0.15) (type solid)) (layer "F.SilkS"))
+    (fp_arc (start -3.75 -2) (mid -3.603553 -2.353553) (end -3.25 -2.5)
+      (stroke (width 0.15) (type solid)) (layer "F.SilkS"))
+    (fp_arc (start -3.25 2.5) (mid -3.603553 2.353553) (end -3.75 2)
+      (stroke (width 0.15) (type solid)) (layer "F.SilkS"))
+    (fp_arc (start 3.25 -2.5) (mid 3.603553 -2.353553) (end 3.75 -2)
+      (stroke (width 0.15) (type solid)) (layer "F.SilkS"))
+    (fp_arc (start 3.75 2) (mid 3.603553 2.353553) (end 3.25 2.5)
+      (stroke (width 0.15) (type solid)) (layer "F.SilkS"))
+    (fp_rect (start -3.8 -2.55) (end 3.8 2.6)
+      (stroke (width 0.05) (type solid)) (fill none) (layer "B.CrtYd"))
+    (fp_line (start -4.3 -3) (end -4.3 3)
       (stroke (width 0.025) (type solid)) (layer "F.CrtYd"))
-    (fp_line (start -4 3) (end 4 3)
+    (fp_line (start -4.3 3) (end 4.3 3)
       (stroke (width 0.025) (type solid)) (layer "F.CrtYd"))
-    (fp_line (start 4 -3) (end -4 -3)
+    (fp_line (start 4.3 -3) (end -4.3 -3)
       (stroke (width 0.025) (type solid)) (layer "F.CrtYd"))
-    (fp_line (start 4 3) (end 4 -3)
+    (fp_line (start 4.3 3) (end 4.3 -3)
       (stroke (width 0.025) (type solid)) (layer "F.CrtYd"))
+    (fp_rect (start -3 -2) (end 3 2)
+      (stroke (width 0.1) (type solid)) (fill none) (layer "B.Fab"))
     (pad "1" thru_hole circle (at -2.5 0) (size 1.5 1.5) (drill 1) (layers "*.Cu" "*.Mask")
       (net 1 "Net-(J4-Pin_1)") (pintype "passive"))
+    (pad "1" smd roundrect (at -2 0) (size 3 4.5) (layers "B.Cu" "B.Paste" "B.Mask") (roundrect_rratio 0.1)
+      (net 1 "Net-(J4-Pin_1)") (pintype "passive"))
+    (pad "2" smd roundrect (at 2 0) (size 3 4.5) (layers "B.Cu" "B.Paste" "B.Mask") (roundrect_rratio 0.1)
+      (net 2 "Net-(J8-Pin_1)") (pintype "passive"))
     (pad "2" thru_hole circle (at 2.5 0) (size 1.5 1.5) (drill 1) (layers "*.Cu" "*.Mask")
       (net 2 "Net-(J8-Pin_1)") (pintype "passive"))
@@
       (rotate (xyz 0 0 0))
     )
+    (model "${KICAD7_3DMODEL_DIR}/Capacitor_SMD.3dshapes/C_2512_6332Metric.step"
+      (offset (xyz 0 0 -1.8))
+      (scale (xyz 1 1 1))
+      (rotate (xyz 180 0 0))
+    )
   )
   (footprint "Package_DIP:DIP-8_W7.62mm_Socket" (layer "F.Cu")
@@
     (descr "8-lead though-hole mounted DIP package, row spacing 7.62 mm (300 mils), Socket")
     (tags "THT DIP DIL PDIP 2.54mm 7.62mm 300mil Socket")
-    (property "Sheetfile" "template_1by3.kicad_sch")
+    (property "Sheetfile" "dual_opamp_normal.kicad_sch")
     (property "Sheetname" "")
     (attr through_hole)
@@
     (descr "Open Source Hardware Symbol")
     (tags "Logo Symbol OSHW")
-    (property "Sheetfile" "template_1by3.kicad_sch")
+    (property "Sheetfile" "dual_opamp_normal.kicad_sch")
     (property "Sheetname" "")
     (attr exclude_from_pos_files)
@@
     (descr "Label for general purpose use")
     (tags "Label")
-    (property "Sheetfile" "template_1by3.kicad_sch")
+    (property "Sheetfile" "dual_opamp_normal.kicad_sch")
     (property "Sheetname" "")
     (attr smd)

Commit message: review changes
Parts:
- N1: value V20240523 -> V20240530
Changed lines of the file:
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@@
         (effects (font (size 1 1) (thickness 0.15)) (justify mirror))
     )
-    (fp_text value "V20240523" (at 0.8 0.1) (layer "B.SilkS")
+    (fp_text value "V20240530" (at 0.8 0.1) (layer "B.SilkS")
         (effects (font (size 0.8 0.8) (thickness 0.15)) (justify mirror))
     )
