File: electronics/dual_opamp_normal/dual_opamp_normal.kicad_sch (KiCad schematic)
At the start: 12 parts, among them J1 OUT1, J2 -IN1, J3 +IN1, J4 V-, J5 +IN2, J6 -IN2, J7 OUT2, J8 V+, U1 opamp_dual_8pin

Commit message: updated symbol/footprint tables
Parts:
- C1: footprint SquantorCapacitor:C-050-050X080-film -> SquantorCapacitor:C-050-050X100-0805-3516-film
Changed lines of the file:
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@@
     )
     (instances
-      (project "template_1by3"
+      (project "dual_opamp_normal"
         (path "/10c72907-d560-44b2-a65d-d12510b462b9"
           (reference "N1") (unit 1)
@@
     )
     (instances
-      (project "template_1by3"
+      (project "dual_opamp_normal"
         (path "/10c72907-d560-44b2-a65d-d12510b462b9"
           (reference "N2") (unit 1)
@@
     (pin "1")
     (instances
-      (project "template_1by3"
+      (project "dual_opamp_normal"
         (path "/10c72907-d560-44b2-a65d-d12510b462b9"
           (reference "J2") (unit 1)
@@
     (pin "1")
     (instances
-      (project "template_1by3"
+      (project "dual_opamp_normal"
         (path "/10c72907-d560-44b2-a65d-d12510b462b9"
           (reference "J1") (unit 1)
@@
     (pin "1")
     (instances
-      (project "template_1by3"
+      (project "dual_opamp_normal"
         (path "/10c72907-d560-44b2-a65d-d12510b462b9"
           (reference "J3") (unit 1)
@@
     (pin "1")
     (instances
-      (project "template_1by3"
+      (project "dual_opamp_normal"
         (path "/10c72907-d560-44b2-a65d-d12510b462b9"
           (reference "J4") (unit 1)
@@
     (pin "1")
     (instances
-      (project "template_1by3"
+      (project "dual_opamp_normal"
         (path "/10c72907-d560-44b2-a65d-d12510b462b9"
           (reference "J5") (unit 1)
@@
     (pin "1")
     (instances
-      (project "template_1by3"
+      (project "dual_opamp_normal"
         (path "/10c72907-d560-44b2-a65d-d12510b462b9"
           (reference "J6") (unit 1)
@@
     (pin "1")
     (instances
-      (project "template_1by3"
+      (project "dual_opamp_normal"
         (path "/10c72907-d560-44b2-a65d-d12510b462b9"
           (reference "J8") (unit 1)
@@
     (pin "1")
     (instances
-      (project "template_1by3"
+      (project "dual_opamp_normal"
         (path "/10c72907-d560-44b2-a65d-d12510b462b9"
           (reference "J7") (unit 1)
@@
     (pin "4")
     (instances
-      (project "template_1by3"
+      (project "dual_opamp_normal"
         (path "/10c72907-d560-44b2-a65d-d12510b462b9"
           (reference "U1") (unit 1)
@@
       (effects (font (size 1.27 1.27)))
     )
-    (property "Footprint" "SquantorCapacitor:C-050-050X080-film" (at 43.18 29.5148 0)
+    (property "Footprint" "SquantorCapacitor:C-050-050X100-0805-3516-film" (at 43.18 29.5148 0)
       (effects (font (size 1.27 1.27)) hide)
     )
@@
     (pin "2")
     (instances
-      (project "template_1by3"
+      (project "dual_opamp_normal"
         (path "/10c72907-d560-44b2-a65d-d12510b462b9"
           (reference "C1") (unit 1)

Commit message: review changes
Parts:
- N1: value V20240523 -> V20240530
Changed lines of the file:
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@@
   (junction (at 29.21 45.72) (diameter 0) (color 0 0 0 0)
+  )
+  (junction (at 29.21 30.48) (diameter 0) (color 0 0 0 0)
   )
   (junction (at 49.53 30.48) (diameter 0) (color 0 0 0 0)
@@
     (stroke (width 0) (type default))
   )
+  (wire (pts (xy 29.21 29.21) (xy 29.21 30.48))
+    (stroke (width 0) (type default))
+  )
   (wire (pts (xy 29.21 30.48) (xy 35.56 30.48))
     (stroke (width 0) (type default))
@@
     (stroke (width 0) (type default))
   )
+  (wire (pts (xy 49.53 29.21) (xy 49.53 30.48))
+    (stroke (width 0) (type default))
+  )
   (wire (pts (xy 49.53 53.34) (xy 52.07 53.34))
     (stroke (width 0) (type default))
@@
       (effects (font (size 1.524 1.524)) (justify left))
     )
-    (property "Value" "V20240523" (at 20.32 189.23 0)
+    (property "Value" "V20240530" (at 20.32 189.23 0)
       (effects (font (size 1.524 1.524)) (justify left))
     )
@@
         )
       )
+    )
+  )
+  (symbol (lib_id "power:PWR_FLAG") (at 29.21 29.21 0) (unit 1)
+    (in_bom yes) (on_board yes) (dnp no) (fields_autoplaced)
+    (property "Reference" "#FLG01" (at 29.21 27.305 0)
+      (effects (font (size 1.27 1.27)) hide)
+    )
+    (property "Value" "PWR_FLAG" (at 29.21 24.13 0)
+      (effects (font (size 1.27 1.27)))
+    )
+    (property "Footprint" "" (at 29.21 29.21 0)
+      (effects (font (size 1.27 1.27)) hide)
+    )
+    (property "Datasheet" "~" (at 29.21 29.21 0)
+      (effects (font (size 1.27 1.27)) hide)
+    )
+    (pin "1")
+    (instances
+      (project "dual_opamp_normal"
+        (path "/10c72907-d560-44b2-a65d-d12510b462b9"
+          (reference "#FLG01") (unit 1)
+        )
+      )
+    )
+  )
+  (symbol (lib_id "power:PWR_FLAG") (at 49.53 29.21 0) (unit 1)
+    (in_bom yes) (on_board yes) (dnp no) (fields_autoplaced)
+    (property "Reference" "#FLG02" (at 49.53 27.305 0)
+      (effects (font (size 1.27 1.27)) hide)
+    )
+    (property "Value" "PWR_FLAG" (at 49.53 24.13 0)
+      (effects (font (size 1.27 1.27)))
+    )
+    (property "Footprint" "" (at 49.53 29.21 0)
+      (effects (font (size 1.27 1.27)) hide)
+    )
+    (property "Datasheet" "~" (at 49.53 29.21 0)
+      (effects (font (size 1.27 1.27)) hide)
+    )
+    (pin "1")
+    (instances
+      (project "dual_opamp_normal"
+        (path "/10c72907-d560-44b2-a65d-d12510b462b9"
+          (reference "#FLG02") (unit 1)
+        )
+      )
