File: electronics/dual_opamp_normal/dual_opamp_normal_tiled.kicad_pcb (KiCad board)
At the start: 2 copper layers, 97 x 98.5 mm, 120 parts, among them J1 OUT1, J2 -IN1, J3 +IN1, J4 V-, J5 +IN2, J6 -IN2, J7 OUT2, J8 V+, U1 opamp_dual_8pin

Commit message: reduced tiled sizes and some minor changes
Parts:
- removed the C1 at (148.5, 66.5)
- removed the C1 at (129.0, 66.5)
- removed the C1 at (109.5, 66.5)
- removed the C1 at (168.0, 116.0)
- removed the C1 at (187.5, 116.0)
- removed the C1 at (168.0, 66.5)
- removed the C1 at (187.5, 66.5)
- removed the J1 at (180.0, 53.5)
- removed the J1 at (121.5, 53.5)
- removed the J1 at (102.0, 53.5)
- removed the J1 at (180.0, 103.0)
- removed the J1 at (160.5, 103.0)
- removed the J1 at (160.5, 53.5)
- removed the J1 at (141.0, 53.5)
- removed the J2 at (180.0, 118.0)
- removed the J2 at (121.5, 68.5)
- removed the J2 at (160.5, 68.5)
- removed the J2 at (102.0, 68.5)
- removed the J2 at (141.0, 68.5)
- removed the J2 at (160.5, 118.0)
- removed the J2 at (180.0, 68.5)
- removed the J3 at (160.5, 83.5)
- removed the J3 at (180.0, 133.0)
- removed the J3 at (121.5, 83.5)
- removed the J3 at (102.0, 83.5)
- removed the J3 at (160.5, 133.0)
- removed the J3 at (141.0, 83.5)
- removed the J3 at (180.0, 83.5)
- removed the J4 at (160.5, 98.5)
- removed the J4 at (180.0, 98.5)
- removed the J4 at (180.0, 148.0)
- removed the J4 at (121.5, 98.5)
- removed the J4 at (160.5, 148.0)
- removed the J4 at (141.0, 98.5)
- removed the J4 at (102.0, 98.5)
- removed the J5 at (136.5, 98.5)
- removed the J5 at (156.0, 98.5)
- removed the J5 at (195.0, 98.5)
- removed the J5 at (195.0, 148.0)
- removed the J5 at (175.5, 98.5)
- removed the J5 at (117.0, 98.5)
- removed the J5 at (175.5, 148.0)
- removed the J6 at (175.5, 133.0)
- removed the J6 at (156.0, 83.5)
- removed the J6 at (195.0, 133.0)
- removed the J6 at (117.0, 83.5)
- removed the J6 at (136.5, 83.5)
- removed the J6 at (195.0, 83.5)
- removed the J6 at (175.5, 83.5)
- removed the J7 at (175.5, 118.0)
- removed the J7 at (195.0, 68.5)
- removed the J7 at (117.0, 68.5)
- removed the J7 at (175.5, 68.5)
- removed the J7 at (195.0, 118.0)
- removed the J7 at (156.0, 68.5)
- removed the J7 at (136.5, 68.5)
- removed the J8 at (195.0, 53.5)
- removed the J8 at (175.5, 103.0)
- removed the J8 at (136.5, 53.5)
- removed the J8 at (175.5, 53.5)
- removed the J8 at (195.0, 103.0)
- removed the J8 at (117.0, 53.5)
- removed the J8 at (156.0, 53.5)
- removed the N1 at (166.5, 149.0)
- removed the N1 at (147.0, 99.5)
- removed the N1 at (186.0, 149.0)
- removed the N1 at (186.0, 99.5)
- removed the N1 at (108.0, 99.5)
- removed the N1 at (127.5, 99.5)
- removed the N1 at (166.5, 99.5)
- removed the N2 at (128.5, 95.5)
- removed the N2 at (167.5, 145.0)
- removed the N2 at (109.0, 95.5)
- removed the N2 at (148.0, 95.5)
- removed the N2 at (187.0, 145.0)
- removed the N2 at (167.5, 95.5)
- removed the N2 at (187.0, 95.5)
- removed the U1 at (105.7, 72.2)
- removed the U1 at (183.7, 121.7)
- removed the U1 at (144.7, 72.2)
- removed the U1 at (164.2, 121.7)
- removed the U1 at (125.2, 72.2)
- removed the U1 at (164.2, 72.2)
- removed the U1 at (183.7, 72.2)
Routing:
- net Net-(J4-Pin_1): track 372.1 -> 111.6 mm
- net Net-(J8-Pin_1): track 236.0 -> 70.8 mm
- net Net-(J1-Pin_1): track 211.1 -> 63.3 mm
- net Net-(J5-Pin_1): track 210.8 -> 63.2 mm
- net Net-(J2-Pin_1): track 83.3 -> 25.0 mm
- net Net-(J3-Pin_1): track 83.3 -> 25.0 mm
- net Net-(J7-Pin_1): track 83.1 -> 24.9 mm
- net Net-(J6-Pin_1): track 83.1 -> 24.9 mm
Other:
- board size 97 x 98.5 mm -> 58 x 49 mm
