File: electronics/potmeter_normal/potmeter_normal.kicad_pcb (KiCad board)
At the start: 2 copper layers, 19 x 19 mm, 7 parts, among them J1 1, J2 2, J3 4, J4 3

Commit message: small updates and created a panel
Parts:
- J1: value 1 -> W
- J2: value 2 -> R2
- J3: value 4 -> R1
- J4: value 3 -> R2
- N1: value V20240526 -> V20240530
Changed lines of the file:
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@@
   (footprint "mill-max:PC_pin_nail_head_6092" locked (layer "F.Cu")
     (at 142 63)
-    (property "Sheetfile" "potmeter.kicad_sch")
+    (property "Sheetfile" "potmeter_normal.kicad_sch")
     (property "Sheetname" "")
     (property "ki_description" "Generic connector, single row, 01x01, script generated (kicad-library-utils/schlib/autogen/connector/)")
@@
         (effects (font (size 1 1) (thickness 0.15)))
     )
-    (fp_text value "1" (at 2.5 0) (layer "F.SilkS")
+    (fp_text value "W" (at 3 -0.5) (layer "F.SilkS")
         (effects (font (size 2 2) (thickness 0.3)))
     )
@@
   (footprint "mill-max:PC_pin_nail_head_6092" locked (layer "F.Cu")
     (at 142 78)
-    (property "Sheetfile" "potmeter.kicad_sch")
+    (property "Sheetfile" "potmeter_normal.kicad_sch")
     (property "Sheetname" "")
     (property "ki_description" "Generic connector, single row, 01x01, script generated (kicad-library-utils/schlib/autogen/connector/)")
@@
         (effects (font (size 1 1) (thickness 0.15)))
     )
-    (fp_text value "2" (at 2.5 0) (layer "F.SilkS")
+    (fp_text value "R2" (at 3.5 0.5) (layer "F.SilkS")
         (effects (font (size 2 2) (thickness 0.3)))
     )
@@
   (footprint "mill-max:PC_pin_nail_head_6092" locked (layer "F.Cu")
     (at 157 63)
-    (property "Sheetfile" "potmeter.kicad_sch")
+    (property "Sheetfile" "potmeter_normal.kicad_sch")
     (property "Sheetname" "")
     (property "ki_description" "Generic connector, single row, 01x01, script generated (kicad-library-utils/schlib/autogen/connector/)")
@@
         (effects (font (size 1 1) (thickness 0.15)))
     )
-    (fp_text value "4" (at -2.5 0) (layer "F.SilkS")
+    (fp_text value "R1" (at -3.5 -0.5) (layer "F.SilkS")
         (effects (font (size 2 2) (thickness 0.3)))
     )
@@
   (footprint "mill-max:PC_pin_nail_head_6092" locked (layer "F.Cu")
     (at 157 78)
-    (property "Sheetfile" "potmeter.kicad_sch")
+    (property "Sheetfile" "potmeter_normal.kicad_sch")
     (property "Sheetname" "")
     (property "ki_description" "Generic connector, single row, 01x01, script generated (kicad-library-utils/schlib/autogen/connector/)")
@@
         (effects (font (size 1 1) (thickness 0.15)))
     )
-    (fp_text value "3" (at -2.5 0) (layer "F.SilkS")
+    (fp_text value "R2" (at -3.5 0) (layer "F.SilkS") hide
         (effects (font (size 2 2) (thickness 0.3)))
     )
@@
     (descr "Potentiometer, vertical, Piher PT-15-V15, http://www.piher-nacesa.com/pdf/14-PT15v03.pdf")
     (tags "Potentiometer vertical Piher PT-15-V15")
-    (property "Sheetfile" "potmeter.kicad_sch")
+    (property "Sheetfile" "potmeter_normal.kicad_sch")
     (property "Sheetname" "")
     (property "ki_description" "Potentiometer")
@@
     (descr "Label for general purpose use")
     (tags "Label")
-    (property "Sheetfile" "potmeter.kicad_sch")
+    (property "Sheetfile" "potmeter_normal.kicad_sch")
     (property "Sheetname" "")
     (attr smd)
@@
         (effects (font (size 1 1) (thickness 0.15)) (justify mirror))
     )
-    (fp_text value "V20240526" (at 0 0.1) (layer "B.SilkS")
+    (fp_text value "V20240530" (at 0 0.1) (layer "B.SilkS")
         (effects (font (size 0.8 0.8) (thickness 0.15)) (justify mirror))
     )
@@
     (descr "Open Source Hardware Symbol")
     (tags "Logo Symbol OSHW")
-    (property "Sheetfile" "potmeter.kicad_sch")
+    (property "Sheetfile" "potmeter_normal.kicad_sch")
     (property "Sheetname" "")
     (attr exclude_from_pos_files)
