File: electronics/potmeter_normal/potmeter_normal.kicad_sch (KiCad schematic)
At the start: 7 parts, among them J1 1, J2 2, J3 4, J4 3

Commit message: small updates and created a panel
Parts:
- J1: value 1 -> W
- J2: value 2 -> R2
- J3: value 4 -> R1
- J4: value 3 -> R2
- N1: value V20240526 -> V20240530
Changed lines of the file:
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@@
       (effects (font (size 1.524 1.524)) (justify left))
     )
-    (property "Value" "V20240526" (at 20.32 189.23 0)
+    (property "Value" "V20240530" (at 20.32 189.23 0)
       (effects (font (size 1.524 1.524)) (justify left))
     )
@@
     )
     (instances
-      (project "potmeter"
+      (project "potmeter_normal"
         (path "/b8c0e900-6fea-4c90-a623-0efa02d854c2"
           (reference "N1") (unit 1)
@@
     )
     (instances
-      (project "potmeter"
+      (project "potmeter_normal"
         (path "/b8c0e900-6fea-4c90-a623-0efa02d854c2"
           (reference "N2") (unit 1)
@@
       (effects (font (size 1.27 1.27)))
     )
-    (property "Value" "2" (at 31.75 43.18 0)
+    (property "Value" "R2" (at 31.75 43.18 0)
       (effects (font (size 1.27 1.27)))
     )
@@
     (pin "1")
     (instances
-      (project "potmeter"
+      (project "potmeter_normal"
         (path "/b8c0e900-6fea-4c90-a623-0efa02d854c2"
           (reference "J2") (unit 1)
@@
       (effects (font (size 1.27 1.27)))
     )
-    (property "Value" "1" (at 31.75 33.02 0)
+    (property "Value" "W" (at 31.75 33.02 0)
       (effects (font (size 1.27 1.27)))
     )
@@
     (pin "1")
     (instances
-      (project "potmeter"
+      (project "potmeter_normal"
         (path "/b8c0e900-6fea-4c90-a623-0efa02d854c2"
           (reference "J1") (unit 1)
@@
       (effects (font (size 1.27 1.27)))
     )
-    (property "Value" "4" (at 53.34 33.02 0)
+    (property "Value" "R1" (at 53.34 33.02 0)
       (effects (font (size 1.27 1.27)))
     )
@@
     (pin "1")
     (instances
-      (project "potmeter"
+      (project "potmeter_normal"
         (path "/b8c0e900-6fea-4c90-a623-0efa02d854c2"
           (reference "J3") (unit 1)
@@
       (effects (font (size 1.27 1.27)))
     )
-    (property "Value" "3" (at 53.34 43.18 0)
+    (property "Value" "R2" (at 53.34 43.18 0)
       (effects (font (size 1.27 1.27)))
     )
@@
     (pin "1")
     (instances
-      (project "potmeter"
+      (project "potmeter_normal"
         (path "/b8c0e900-6fea-4c90-a623-0efa02d854c2"
           (reference "J4") (unit 1)
@@
     (pin "3")
     (instances
-      (project "potmeter"
+      (project "potmeter_normal"
         (path "/b8c0e900-6fea-4c90-a623-0efa02d854c2"
           (reference "RV1") (unit 1)
