File: electronics/triple_diode_normal/triple_diode_normal.kicad_pcb (KiCad board)
At the start: 2 copper layers, 19 x 34 mm, 9 parts, among them J1 A1, J2 A2, J3 A3, J4 C3, J5 C2, J6 C1

Commit message: review updates and tiled variant
Parts:
- N1: value V20220113 -> V20240530
Changed lines of the file:
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@@
         (effects (font (size 1 1) (thickness 0.15)) (justify mirror))
     )
-    (fp_text value "V20220113" (at 0 0) (layer "B.SilkS")
+    (fp_text value "V20240530" (at 0 0) (layer "B.SilkS")
         (effects (font (size 0.8 0.8) (thickness 0.15)) (justify mirror))
     )
