File: electronics/triple_diode_normal/triple_diode_normal.kicad_sch (KiCad schematic)
At the start: 9 parts, among them J1 A1, J2 A2, J3 A3, J4 C3, J5 C2, J6 C1

Commit message: review updates and tiled variant
Parts:
- N1: value V20220113 -> V20240530
Changed lines of the file:
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@@
       (effects (font (size 1.524 1.524)) (justify left))
     )
-    (property "Value" "V20220113" (at 20.32 189.23 0)
+    (property "Value" "V20240530" (at 20.32 189.23 0)
       (effects (font (size 1.524 1.524)) (justify left))
     )
