File: electronics/triple_diode_XN/triple_diode_XN.kicad_sch (KiCad schematic)
At the start: 9 parts, among them J1 A1, J2 A2, J3 A3, J4 C3, J5 C2, J6 C1

Commit message: updates and tiled
Parts:
- N1: value V20240506 -> V20240530
Changed lines of the file:
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@@
       (effects (font (size 1.524 1.524)) (justify left))
     )
-    (property "Value" "V20240506" (at 20.32 189.23 0)
+    (property "Value" "V20240530" (at 20.32 189.23 0)
       (effects (font (size 1.524 1.524)) (justify left))
     )
@@
     )
     (instances
-      (project "triple_diode_normal"
+      (project "triple_diode_XN"
         (path "/4afa80ff-4542-4837-ba2e-ef55b455ed28"
           (reference "N1") (unit 1)
@@
     )
     (instances
-      (project "triple_diode_normal"
+      (project "triple_diode_XN"
         (path "/4afa80ff-4542-4837-ba2e-ef55b455ed28"
           (reference "N2") (unit 1)
@@
     (pin "1")
     (instances
-      (project "triple_diode_normal"
+      (project "triple_diode_XN"
         (path "/4afa80ff-4542-4837-ba2e-ef55b455ed28"
           (reference "J2") (unit 1)
@@
     (pin "1")
     (instances
-      (project "triple_diode_normal"
+      (project "triple_diode_XN"
         (path "/4afa80ff-4542-4837-ba2e-ef55b455ed28"
           (reference "J1") (unit 1)
@@
     (pin "1")
     (instances
-      (project "triple_diode_normal"
+      (project "triple_diode_XN"
         (path "/4afa80ff-4542-4837-ba2e-ef55b455ed28"
           (reference "J3") (unit 1)
@@
     (pin "1")
     (instances
-      (project "triple_diode_normal"
+      (project "triple_diode_XN"
         (path "/4afa80ff-4542-4837-ba2e-ef55b455ed28"
           (reference "J4") (unit 1)
@@
     (pin "1")
     (instances
-      (project "triple_diode_normal"
+      (project "triple_diode_XN"
         (path "/4afa80ff-4542-4837-ba2e-ef55b455ed28"
           (reference "J5") (unit 1)
@@
     (pin "1")
     (instances
-      (project "triple_diode_normal"
+      (project "triple_diode_XN"
         (path "/4afa80ff-4542-4837-ba2e-ef55b455ed28"
           (reference "J6") (unit 1)
@@
     (pin "5")
     (instances
-      (project "triple_diode_normal"
+      (project "triple_diode_XN"
         (path "/4afa80ff-4542-4837-ba2e-ef55b455ed28"
           (reference "D1") (unit 1)
