File: electronics/triple_diode_XN/triple_diode_XN.kicad_pcb (KiCad board)
At the start: 2 copper layers, 19 x 19 mm, 9 parts, among them J1 A1, J2 A2, J3 A3, J4 C3, J5 C2, J6 C1

Commit message: updates and tiled
Parts:
- N1: value V20240506 -> V20240530
Changed lines of the file:
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@@
         (effects (font (size 1 1) (thickness 0.15)) (justify mirror))
     )
-    (fp_text value "V20240506" (at 0 0.1) (layer "B.SilkS")
+    (fp_text value "V20240530" (at 0 0.1) (layer "B.SilkS")
         (effects (font (size 0.8 0.8) (thickness 0.15)) (justify mirror))
     )

Commit message: reduced tiled sizes and some minor changes
Changed lines of the file:
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@@
   (gr_line (start 148 62.5) (end 152 62.5)
     (stroke (width 0.3) (type default)) (layer "F.SilkS"))
-  (gr_rect (start 142.5 72) (end 157.5 75.5)
-    (stroke (width 0.3) (type solid)) (fill solid) (layer "F.SilkS"))
   (gr_poly
     (pts
