File: electronics/triple_diode_XN/triple_diode_XN_tiled.kicad_pcb (KiCad board)
At the start: 2 copper layers, 77.5 x 77.5 mm, 144 parts, among them J1 A1, J2 A2, J3 A3, J4 C3, J5 C2, J6 C1

Commit message: reduced tiled sizes and some minor changes
Parts:
- removed the D1 at (118.0, 121.0)
- removed the D1 at (118.0, 101.5)
- removed the D1 at (118.0, 82.0)
- removed the D1 at (118.0, 140.5)
- removed the D1 at (79.0, 82.0)
- removed the D1 at (59.5, 82.0)
- removed the D1 at (98.5, 82.0)
- removed the J1 at (91.0, 74.5)
- removed the J1 at (110.5, 74.5)
- removed the J1 at (110.5, 113.5)
- removed the J1 at (52.0, 74.5)
- removed the J1 at (71.5, 74.5)
- removed the J1 at (110.5, 133.0)
- removed the J1 at (110.5, 94.0)
- removed the J2 at (71.5, 82.0)
- removed the J2 at (91.0, 82.0)
- removed the J2 at (110.5, 121.0)
- removed the J2 at (110.5, 140.5)
- removed the J2 at (52.0, 82.0)
- removed the J2 at (110.5, 101.5)
- removed the J2 at (110.5, 82.0)
- removed the J3 at (91.0, 89.5)
- removed the J3 at (52.0, 89.5)
- removed the J3 at (110.5, 128.5)
- removed the J3 at (110.5, 109.0)
- removed the J3 at (110.5, 148.0)
- removed the J3 at (110.5, 89.5)
- removed the J3 at (71.5, 89.5)
- removed the J4 at (125.5, 148.0)
- removed the J4 at (106.0, 89.5)
- removed the J4 at (86.5, 89.5)
- removed the J4 at (125.5, 89.5)
- removed the J4 at (125.5, 109.0)
- removed the J4 at (67.0, 89.5)
- removed the J4 at (125.5, 128.5)
- removed the J5 at (125.5, 121.0)
- removed the J5 at (125.5, 101.5)
- removed the J5 at (86.5, 82.0)
- removed the J5 at (125.5, 82.0)
- removed the J5 at (106.0, 82.0)
- removed the J5 at (125.5, 140.5)
- removed the J5 at (67.0, 82.0)
- removed the J6 at (86.5, 74.5)
- removed the J6 at (125.5, 133.0)
- removed the J6 at (106.0, 74.5)
- removed the J6 at (125.5, 94.0)
- removed the J6 at (67.0, 74.5)
- removed the J6 at (125.5, 113.5)
- removed the J6 at (125.5, 74.5)
- removed the N1 at (118.0, 104.0)
- removed the N1 at (98.5, 84.5)
- removed the N1 at (59.5, 84.5)
- removed the N1 at (118.0, 84.5)
- removed the N1 at (118.0, 143.0)
- removed the N1 at (79.0, 84.5)
- removed the N1 at (118.0, 123.5)
- removed the N2 at (118.0, 139.5)
- removed the N2 at (118.0, 100.5)
- removed the N2 at (118.0, 120.0)
- removed the N2 at (79.0, 81.0)
- removed the N2 at (98.5, 81.0)
- removed the N2 at (59.5, 81.0)
- removed the N2 at (118.0, 81.0)
Routing:
- net Net-(D1-A1): track 202.3 -> 113.8 mm, vias 16 -> 9
- net Net-(D1-C3): track 202.3 -> 113.8 mm, vias 16 -> 9
- net Net-(D1-C1): track 202.3 -> 113.8 mm, vias 16 -> 9
- net Net-(D1-A3): track 202.3 -> 113.8 mm, vias 16 -> 9
- net Net-(D1-C2): track 103.2 -> 58.1 mm, vias 16 -> 9
- net Net-(D1-A2): track 103.2 -> 58.1 mm, vias 16 -> 9
Other:
- board size 77.5 x 77.5 mm -> 58 x 58 mm
