File: electronics/transistor_SOT23/transistor_SOT23.kicad_pcb (KiCad board)
At the start: 2 copper layers, 19 x 19 mm, 7 parts, among them J1 B or G, J2 E or S, J3 C or D, J4 E or S, Q1 Q_NPN_BEC

Commit message: updated versionnumber location
Parts:
- moved N1 0.75 mm to (157.2, 71.5)
Changed lines of the file:
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@@
       (effects (font (size 1 1) (thickness 0.15)))
     )
+    (fp_line (start -1.2 -0.2) (end 1.2 -0.2) (layer F.SilkS) (width 0.15))
+    (fp_line (start 1.2 -0.2) (end 1.2 0.2) (layer F.SilkS) (width 0.15))
+    (fp_line (start 1.2 0.2) (end -1.2 0.2) (layer F.SilkS) (width 0.15))
+    (fp_line (start -1.2 0.2) (end -1.2 -0.2) (layer F.SilkS) (width 0.15))
+    (fp_line (start -1.7 1.8) (end 1.7 1.8) (layer F.CrtYd) (width 0.05))
+    (fp_line (start -1.7 1.8) (end -1.7 -1.1) (layer F.CrtYd) (width 0.05))
+    (fp_line (start -1.7 -1.1) (end -0.7 -1.1) (layer F.CrtYd) (width 0.05))
+    (fp_line (start -0.7 -1.1) (end -0.7 -1.8) (layer F.CrtYd) (width 0.05))
+    (fp_line (start -0.7 -1.8) (end 0.7 -1.8) (layer F.CrtYd) (width 0.05))
+    (fp_line (start 0.7 -1.8) (end 0.7 -1.1) (layer F.CrtYd) (width 0.05))
+    (fp_line (start 0.7 -1.1) (end 1.7 -1.1) (layer F.CrtYd) (width 0.05))
     (fp_line (start 1.7 -1.1) (end 1.7 1.8) (layer F.CrtYd) (width 0.05))
-    (fp_line (start 0.7 -1.1) (end 1.7 -1.1) (layer F.CrtYd) (width 0.05))
-    (fp_line (start 0.7 -1.8) (end 0.7 -1.1) (layer F.CrtYd) (width 0.05))
-    (fp_line (start -0.7 -1.8) (end 0.7 -1.8) (layer F.CrtYd) (width 0.05))
-    (fp_line (start -0.7 -1.1) (end -0.7 -1.8) (layer F.CrtYd) (width 0.05))
-    (fp_line (start -1.7 -1.1) (end -0.7 -1.1) (layer F.CrtYd) (width 0.05))
-    (fp_line (start -1.7 1.8) (end -1.7 -1.1) (layer F.CrtYd) (width 0.05))
-    (fp_line (start -1.7 1.8) (end 1.7 1.8) (layer F.CrtYd) (width 0.05))
-    (fp_line (start -1.2 0.2) (end -1.2 -0.2) (layer F.SilkS) (width 0.15))
-    (fp_line (start 1.2 0.2) (end -1.2 0.2) (layer F.SilkS) (width 0.15))
-    (fp_line (start 1.2 -0.2) (end 1.2 0.2) (layer F.SilkS) (width 0.15))
-    (fp_line (start -1.2 -0.2) (end 1.2 -0.2) (layer F.SilkS) (width 0.15))
     (pad 3 smd rect (at 0 -1 270) (size 0.8 0.9) (layers F.Cu F.Paste F.Mask)
       (net 3 /C) (zone_connect 2))
@@
       (effects (font (size 1 1) (thickness 0.15)))
     )
+    (fp_circle (center 0 0) (end 1.3 0) (layer F.CrtYd) (width 0.025))
     (fp_circle (center 0 0) (end 1.3 0) (layer B.CrtYd) (width 0.025))
-    (fp_circle (center 0 0) (end 1.3 0) (layer F.CrtYd) (width 0.025))
     (pad 1 thru_hole circle (at 0 0) (size 2 2) (drill 1.1) (layers *.Cu *.Mask)
       (net 2 /E))
@@
       (effects (font (size 1 1) (thickness 0.15)))
     )
+    (fp_circle (center 0 0) (end 1.3 0) (layer F.CrtYd) (width 0.025))
     (fp_circle (center 0 0) (end 1.3 0) (layer B.CrtYd) (width 0.025))
-    (fp_circle (center 0 0) (end 1.3 0) (layer F.CrtYd) (width 0.025))
     (pad 1 thru_hole circle (at 0 0) (size 2 2) (drill 1.1) (layers *.Cu *.Mask)
       (net 3 /C))
@@
       (effects (font (size 1 1) (thickness 0.15)))
     )
+    (fp_circle (center 0 0) (end 1.3 0) (layer F.CrtYd) (width 0.025))
     (fp_circle (center 0 0) (end 1.3 0) (layer B.CrtYd) (width 0.025))
-    (fp_circle (center 0 0) (end 1.3 0) (layer F.CrtYd) (width 0.025))
     (pad 1 thru_hole circle (at 0 0) (size 2 2) (drill 1.1) (layers *.Cu *.Mask)
       (net 2 /E))
@@
       (effects (font (size 1 1) (thickness 0.15)))
     )
+    (fp_circle (center 0 0) (end 1.3 0) (layer F.CrtYd) (width 0.025))
     (fp_circle (center 0 0) (end 1.3 0) (layer B.CrtYd) (width 0.025))
-    (fp_circle (center 0 0) (end 1.3 0) (layer F.CrtYd) (width 0.025))
     (pad 1 thru_hole circle (at 0 0) (size 2 2) (drill 1.1) (layers *.Cu *.Mask)
       (net 1 /B))
@@
   )
   (module SquantorLabels:Label_Generic (layer B.Cu)
-    (at 157.25 70.75 90)
+    (at 157.25 71.5 90)
     (descr "Label for general purpose use")
     (tags Label)

Commit message: updated versionnumber, small schematic fixes
Parts:
- N1: value V20201122 -> V20201127
Changed lines of the file:
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@@
       (effects (font (size 1 1) (thickness 0.15)))
     )
+    (fp_line (start 1.7 -1.1) (end 1.7 1.8) (layer F.CrtYd) (width 0.05))
+    (fp_line (start 0.7 -1.1) (end 1.7 -1.1) (layer F.CrtYd) (width 0.05))
+    (fp_line (start 0.7 -1.8) (end 0.7 -1.1) (layer F.CrtYd) (width 0.05))
+    (fp_line (start -0.7 -1.8) (end 0.7 -1.8) (layer F.CrtYd) (width 0.05))
+    (fp_line (start -0.7 -1.1) (end -0.7 -1.8) (layer F.CrtYd) (width 0.05))
+    (fp_line (start -1.7 -1.1) (end -0.7 -1.1) (layer F.CrtYd) (width 0.05))
+    (fp_line (start -1.7 1.8) (end -1.7 -1.1) (layer F.CrtYd) (width 0.05))
+    (fp_line (start -1.7 1.8) (end 1.7 1.8) (layer F.CrtYd) (width 0.05))
+    (fp_line (start -1.2 0.2) (end -1.2 -0.2) (layer F.SilkS) (width 0.15))
+    (fp_line (start 1.2 0.2) (end -1.2 0.2) (layer F.SilkS) (width 0.15))
+    (fp_line (start 1.2 -0.2) (end 1.2 0.2) (layer F.SilkS) (width 0.15))
     (fp_line (start -1.2 -0.2) (end 1.2 -0.2) (layer F.SilkS) (width 0.15))
-    (fp_line (start 1.2 -0.2) (end 1.2 0.2) (layer F.SilkS) (width 0.15))
-    (fp_line (start 1.2 0.2) (end -1.2 0.2) (layer F.SilkS) (width 0.15))
-    (fp_line (start -1.2 0.2) (end -1.2 -0.2) (layer F.SilkS) (width 0.15))
-    (fp_line (start -1.7 1.8) (end 1.7 1.8) (layer F.CrtYd) (width 0.05))
-    (fp_line (start -1.7 1.8) (end -1.7 -1.1) (layer F.CrtYd) (width 0.05))
-    (fp_line (start -1.7 -1.1) (end -0.7 -1.1) (layer F.CrtYd) (width 0.05))
-    (fp_line (start -0.7 -1.1) (end -0.7 -1.8) (layer F.CrtYd) (width 0.05))
-    (fp_line (start -0.7 -1.8) (end 0.7 -1.8) (layer F.CrtYd) (width 0.05))
-    (fp_line (start 0.7 -1.8) (end 0.7 -1.1) (layer F.CrtYd) (width 0.05))
-    (fp_line (start 0.7 -1.1) (end 1.7 -1.1) (layer F.CrtYd) (width 0.05))
-    (fp_line (start 1.7 -1.1) (end 1.7 1.8) (layer F.CrtYd) (width 0.05))
     (pad 3 smd rect (at 0 -1 270) (size 0.8 0.9) (layers F.Cu F.Paste F.Mask)
       (net 3 /C) (zone_connect 2))
@@
       (effects (font (size 1 1) (thickness 0.15)))
     )
+    (fp_circle (center 0 0) (end 1.3 0) (layer B.CrtYd) (width 0.025))
     (fp_circle (center 0 0) (end 1.3 0) (layer F.CrtYd) (width 0.025))
-    (fp_circle (center 0 0) (end 1.3 0) (layer B.CrtYd) (width 0.025))
     (pad 1 thru_hole circle (at 0 0) (size 2 2) (drill 1.1) (layers *.Cu *.Mask)
       (net 2 /E))
@@
       (effects (font (size 1 1) (thickness 0.15)))
     )
+    (fp_circle (center 0 0) (end 1.3 0) (layer B.CrtYd) (width 0.025))
     (fp_circle (center 0 0) (end 1.3 0) (layer F.CrtYd) (width 0.025))
-    (fp_circle (center 0 0) (end 1.3 0) (layer B.CrtYd) (width 0.025))
     (pad 1 thru_hole circle (at 0 0) (size 2 2) (drill 1.1) (layers *.Cu *.Mask)
       (net 3 /C))
@@
       (effects (font (size 1 1) (thickness 0.15)))
     )
+    (fp_circle (center 0 0) (end 1.3 0) (layer B.CrtYd) (width 0.025))
     (fp_circle (center 0 0) (end 1.3 0) (layer F.CrtYd) (width 0.025))
-    (fp_circle (center 0 0) (end 1.3 0) (layer B.CrtYd) (width 0.025))
     (pad 1 thru_hole circle (at 0 0) (size 2 2) (drill 1.1) (layers *.Cu *.Mask)
       (net 2 /E))
@@
       (effects (font (size 1 1) (thickness 0.15)))
     )
+    (fp_circle (center 0 0) (end 1.3 0) (layer B.CrtYd) (width 0.025))
     (fp_circle (center 0 0) (end 1.3 0) (layer F.CrtYd) (width 0.025))
-    (fp_circle (center 0 0) (end 1.3 0) (layer B.CrtYd) (width 0.025))
     (pad 1 thru_hole circle (at 0 0) (size 2 2) (drill 1.1) (layers *.Cu *.Mask)
       (net 1 /B))
@@
       (effects (font (size 1 1) (thickness 0.15)) (justify mirror))
     )
-    (fp_text value V20201122 (at 0.8 0.1 90) (layer B.SilkS)
+    (fp_text value V20201127 (at 0.8 0.1 90) (layer B.SilkS)
       (effects (font (size 0.8 0.8) (thickness 0.15)) (justify mirror))
     )

Commit message: updated to newer version
Other:
- net class Default removed
- rule pad_to_mask_clearance: 0.0762 -> 0

Commit message: review updates, added tiled version
Parts:
- N1: value V20201127 -> V20240530
- turned Q1 to 0 degrees
