File: electronics/transistor_SOT23/transistor_SOT23.kicad_sch (KiCad schematic)
At the start: 7 parts, among them J1 B or G, J2 E or S, J3 C or D, J4 E or S, Q1 Q_NPN_BEC

Commit message: review updates, added tiled version
Parts:
- N1: value V20201127 -> V20240530
Changed lines of the file:
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@@
     (effects (font (size 1.27 1.27)) (justify left bottom))
   )
-  (label "E" (at 40.64 46.99 0)
+  (label "E" (at 40.64 46.99 0) (fields_autoplaced)
     (effects (font (size 1.27 1.27)) (justify left bottom))
   )
-  (label "C" (at 44.45 30.48 0)
+  (label "C" (at 44.45 30.48 0) (fields_autoplaced)
     (effects (font (size 1.27 1.27)) (justify left bottom))
   )
-  (label "B" (at 35.56 30.48 0)
+  (label "B" (at 35.56 30.48 0) (fields_autoplaced)
     (effects (font (size 1.27 1.27)) (justify left bottom))
   )
@@
       (effects (font (size 1.524 1.524)) (justify left))
     )
-    (property "Value" "V20201127" (at 20.32 189.23 0)
+    (property "Value" "V20240530" (at 20.32 189.23 0)
       (effects (font (size 1.524 1.524)) (justify left))
     )
